Commit message: pt E final (post submission) but with correct joints

File: body.urdf (robot description, URDF)
Before this commit: robot robot, 3 links, 2 joints
Joints:
- joint torso_backleg: origin xyz=0 2.5 1.5 rpy=0 0 0 -> xyz=2.5 0 1.5 rpy=0 0 0
- joint torso_frontleg: origin xyz=0 1.5 1.5 rpy=0 0 0 -> xyz=1.5 0 1.5 rpy=0 0 0

Commit message: pt G openloop control of movement

File: body.urdf (robot description, URDF)
Before this commit: robot robot, 3 links, 2 joints
Joints:
- joint torso_backleg: origin xyz=2.5 0 1.5 rpy=0 0 0 -> xyz=2 0 1 rpy=0 0 0
- joint torso_frontleg: origin xyz=1.5 0 1.5 rpy=0 0 0 -> xyz=1 0 1 rpy=0 0 0

Commit message: pt N changing joint axes complete

File: body.urdf (robot description, URDF)
Before this commit: robot robot, 3 links, 2 joints
Joints:
- joint torso_backleg: axis 0 1 0 -> 1 0 0
- joint torso_frontleg: axis 0 1 0 -> 1 0 0

Commit message: pt N workign through the lower legs

File: body.urdf (robot description, URDF)
Before this commit: robot robot, 3 links, 2 joints
Links:
- added link backlowerleg, mass 1; collision box size=0.2 0.2 1; visual box size=0.2 0.2 1
- added link frontlowerleg, mass 1; collision box size=0.2 0.2 1; visual box size=0.2 0.2 1
- added link leftleg, mass 1; collision box size=1 0.2 0.2; visual box size=1 0.2 0.2
- added link leftlowerleg, mass 1; collision box size=0.2 0.2 1; visual box size=0.2 0.2 1
- added link rightleg, mass 1; collision box size=1 0.2 0.2; visual box size=1 0.2 0.2
- added link rightlowerleg, mass 1; collision box size=0.2 0.2 1; visual box size=0.2 0.2 1
Joints:
- added joint backleg_backlowerleg: type revolute, parent torso, child backlowerleg, origin xyz=0 -1 0 rpy=0 0 0, axis 1 0 0, limit lower=-3.14159 upper=3.14159 effort=0.0 velocity=0.0
- added joint front_frontlowerleg: type revolute, parent torso, child frontlowerleg, origin xyz=0 1 0 rpy=0 0 0, axis 1 0 0, limit lower=-3.14159 upper=3.14159 effort=0.0 velocity=0.0
- added joint leftleg_leftlowerleg: type revolute, parent torso, child leftlowerleg, origin xyz=-1 0 0 rpy=0 0 0, axis 0 1 0, limit lower=-3.14159 upper=3.14159 effort=0.0 velocity=0.0
- added joint rightleg_rightlowerleg: type revolute, parent torso, child rightlowerleg, origin xyz=1 0 0 rpy=0 0 0, axis 0 1 0, limit lower=-3.14159 upper=3.14159 effort=0.0 velocity=0.0
- added joint torso_leftleg: type revolute, parent torso, child leftleg, origin xyz=-0.5 0 1 rpy=0 0 0, axis 0 1 0, limit lower=-3.14159 upper=3.14159 effort=0.0 velocity=0.0
- added joint torso_rightleg: type revolute, parent torso, child rightleg, origin xyz=0.5 0 1 rpy=0 0 0, axis 0 1 0, limit lower=-3.14159 upper=3.14159 effort=0.0 velocity=0.0

Commit message: pt N lower legs complete

File: body.urdf (robot description, URDF)
Before this commit: robot robot, 9 links, 8 joints
Joints:
- removed joint front_frontlowerleg
- added joint frontleg_frontlowerleg: type revolute, parent frontleg, child frontlowerleg, origin xyz=0 1 0 rpy=0 0 0, axis 0 1 0, limit lower=-3.14159 upper=3.14159 effort=0.0 velocity=0.0
- joint backleg_backlowerleg: axis 1 0 0 -> 0 1 0; parent torso -> backleg
- joint leftleg_leftlowerleg: parent torso -> leftleg
- joint rightleg_rightlowerleg: parent torso -> rightleg

Commit message: ass5: added golfer and course

File: body.urdf (robot description, URDF)
Before this commit: robot robot, 9 links, 8 joints
Links:
- removed link backleg
- removed link backlowerleg
- removed link frontleg
- removed link frontlowerleg
- removed link leftleg
- removed link leftlowerleg
- removed link rightleg
- removed link rightlowerleg
- added link arm, mass 1; collision box size=0.3333333333333333 2.5 0.3333333333333333; visual box size=0.3333333333333333 2.5 0.3333333333333333
- added link club, mass 1; collision box size=0.3333333333333333 0.3333333333333333 2.5; visual box size=0.3333333333333333 0.3333333333333333 2.5
- link torso: geometry collision box size=1 1 3; visual box size=1 1 3
Joints:
- removed joint backleg_backlowerleg
- removed joint frontleg_frontlowerleg
- removed joint leftleg_leftlowerleg
- removed joint rightleg_rightlowerleg
- removed joint torso_backleg
- removed joint torso_frontleg
- removed joint torso_leftleg
- removed joint torso_rightleg
- added joint arm_club: type fixed, parent arm, child club, origin xyz=0 2.5 0 rpy=0 0 0, axis 1 0 0, limit lower=-3.14159 upper=3.14159 effort=0.0 velocity=0.0
- added joint torso_arm: type revolute, parent torso, child arm, origin xyz=0 -2.5 4 rpy=0 0 0, axis 0 1 0, limit lower=-3.14159 upper=3.14159 effort=0.0 velocity=0.0

Commit message: ass5 adjusted URDF so robot links could have mass adjustments

File: body.urdf (robot description, URDF)
Before this commit: robot robot, 3 links, 2 joints
Links:
- link arm: mass 1 -> 1.0
- link club: mass 1 -> 1.0
- link torso: mass 1 -> 1000.0

Commit message: ass5 all prepped to add in "state of the world" and then to program fitness

File: body.urdf (robot description, URDF)
Before this commit: robot robot, 3 links, 2 joints
Links:
- link club: geometry collision box size=0.3333333333333333 0.3333333333333333 2.8; visual box size=0.3333333333333333 0.3333333333333333 2.8
- link torso: mass 1000.0 -> 10000.0

Commit message: ass5 added hip joint

File: body.urdf (robot description, URDF)
Before this commit: robot robot, 3 links, 2 joints
Links:
- added link hip, mass 10000.0; collision box size=1 1 0.5; visual box size=1 1 0.5
- link torso: mass 10000.0 -> 1000.0
Joints:
- added joint torso_hip: type revolute, parent torso, child hip, origin xyz=0 -3 1.75 rpy=0 0 0, axis 0 0 1, limit lower=-3.14159 upper=3.14159 effort=0.0 velocity=0.0

Commit message: ass6: making progress

File: body.urdf (robot description, URDF)
Before this commit: robot robot, 4 links, 3 joints
Links:
- removed link arm
- removed link club
- removed link hip
- removed link torso
- added link rootLink, mass 1.0; collision box size=1 1 1; visual box size=1 1 1
Joints:
- removed joint arm_club
- removed joint torso_arm
- removed joint torso_hip

Commit message: ass6: created random links, random joints, and if statement for color

File: body.urdf (robot description, URDF)
Before this commit: robot robot, 1 links, 0 joints
Links:
- added link link1, mass 3.601672253946525; collision box size=0.7349747131998585 1.8184446944008248 2.0962970320876266; visual box size=0.7349747131998585 1.8184446944008248 2.0962970320876266
- added link link10, mass 0.456035290372524; collision box size=1.0577457102017553 1.1138885853087543 2.436674168405964; visual box size=1.0577457102017553 1.1138885853087543 2.436674168405964
- added link link2, mass 4.86086328798975; collision box size=0.976531988691246 1.8425088524037847 0.8059763025935918; visual box size=0.976531988691246 1.8425088524037847 0.8059763025935918
- added link link3, mass 3.45707287010687; collision box size=1.2517540676601264 1.8723554867331458 2.08456887183416; visual box size=1.2517540676601264 1.8723554867331458 2.08456887183416
- added link link4, mass 4.318607293010379; collision box size=2.4295077829422462 1.143559907168321 1.8371572983025675; visual box size=2.4295077829422462 1.143559907168321 1.8371572983025675
- added link link5, mass 1.4501330092957891; collision box size=1.5520066356970015 2.2400611967658843 0.6897474884252648; visual box size=1.5520066356970015 2.2400611967658843 0.6897474884252648
- added link link6, mass 2.18725981529122; collision box size=1.6191688742315353 2.2120139522122386 0.8738310292456029; visual box size=1.6191688742315353 2.2120139522122386 0.8738310292456029
- added link link7, mass 0.6755047916301982; collision box size=1.0198209073447824 1.1006250895846477 1.439095005046205; visual box size=1.0198209073447824 1.1006250895846477 1.439095005046205
- added link link8, mass 3.483822411530411; collision box size=2.2164977877440064 2.4011052142386333 1.2104463865479191; visual box size=2.2164977877440064 2.4011052142386333 1.2104463865479191
- added link link9, mass 4.9015760334571254; collision box size=1.0577457102017553 0.5934318280589641 1.2818486919568717; visual box size=1.0577457102017553 0.5934318280589641 1.2818486919568717
Joints:
- added joint link1_link2: type revolute, parent link1, child link2, origin xyz=0.7349747131998585 0 0 rpy=0 0 0, axis 0 1 0, limit lower=-3.14159 upper=3.14159 effort=0.0 velocity=0.0
- added joint link2_link3: type revolute, parent link2, child link3, origin xyz=0.976531988691246 0 0 rpy=0 0 0, axis 0 1 0, limit lower=-3.14159 upper=3.14159 effort=0.0 velocity=0.0
- added joint link3_link4: type revolute, parent link3, child link4, origin xyz=1.2517540676601264 0 0 rpy=0 0 0, axis 0 1 0, limit lower=-3.14159 upper=3.14159 effort=0.0 velocity=0.0
- added joint link4_link5: type revolute, parent link4, child link5, origin xyz=2.4295077829422462 0 0 rpy=0 0 0, axis 0 1 0, limit lower=-3.14159 upper=3.14159 effort=0.0 velocity=0.0
- added joint link5_link6: type revolute, parent link5, child link6, origin xyz=1.5520066356970015 0 0 rpy=0 0 0, axis 0 1 0, limit lower=-3.14159 upper=3.14159 effort=0.0 velocity=0.0
- added joint link6_link7: type revolute, parent link6, child link7, origin xyz=1.6191688742315353 0 0 rpy=0 0 0, axis 0 1 0, limit lower=-3.14159 upper=3.14159 effort=0.0 velocity=0.0
- added joint link7_link8: type revolute, parent link7, child link8, origin xyz=1.0198209073447824 0 0 rpy=0 0 0, axis 0 1 0, limit lower=-3.14159 upper=3.14159 effort=0.0 velocity=0.0
- added joint link8_link9: type revolute, parent link8, child link9, origin xyz=2.2164977877440064 0 0 rpy=0 0 0, axis 0 1 0, limit lower=-3.14159 upper=3.14159 effort=0.0 velocity=0.0
- added joint link9_link10: type revolute, parent link9, child link10, origin xyz=1.0577457102017553 0 0 rpy=0 0 0, axis 0 1 0, limit lower=-3.14159 upper=3.14159 effort=0.0 velocity=0.0
- added joint rootLink_link1: type revolute, parent rootLink, child link1, origin xyz=0.5 0 6 rpy=0 0 0, axis 0 1 0, limit lower=-3.14159 upper=3.14159 effort=0.0 velocity=0.0

Commit message: ass6: figuring out how to add neurons to randomized snake

File: body.urdf (robot description, URDF)
Before this commit: robot robot, 11 links, 10 joints
Links:
- removed link link10
- removed link link8
- removed link link9
- removed link rootLink
- link link1: mass 3.601672253946525 -> 3.798663505993619; geometry collision box size=2.1681310979844666 1.9546504833205403 1.6532021905903542; visual box size=2.1681310979844666 1.9546504833205403 1.6532021905903542
- link link2: mass 4.86086328798975 -> 0.1042664700510676; geometry collision box size=0.5584553558758178 0.809321799051185 1.4144910667436301; visual box size=0.5584553558758178 0.809321799051185 1.4144910667436301
- link link3: mass 3.45707287010687 -> 0.9388419124094066; geometry collision box size=2.1055454153171325 2.340374676602882 2.064797751797774; visual box size=2.1055454153171325 2.340374676602882 2.064797751797774
- link link4: mass 4.318607293010379 -> 0.2421340325638499; geometry collision box size=1.093697705160728 0.7902872201787827 0.8439647615053572; visual box size=1.093697705160728 0.7902872201787827 0.8439647615053572
- link link5: mass 1.4501330092957891 -> 2.1958066847564286; geometry collision box size=1.3719094999863397 2.2663414371984967 2.2124868282407038; visual box size=1.3719094999863397 2.2663414371984967 2.2124868282407038
- link link6: mass 2.18725981529122 -> 4.329982891495016; geometry collision box size=1.2043036478969262 0.5738860312233407 2.3806809013379606; visual box size=1.2043036478969262 0.5738860312233407 2.3806809013379606
- link link7: mass 0.6755047916301982 -> 4.522658602844529; geometry collision box size=1.2043036478969262 2.4357945867911006 2.1671053491001846; visual box size=1.2043036478969262 2.4357945867911006 2.1671053491001846
Joints:
- removed joint link7_link8
- removed joint link8_link9
- removed joint link9_link10
- removed joint rootLink_link1
- joint link1_link2: origin xyz=0.7349747131998585 0 0 rpy=0 0 0 -> xyz=2.1681310979844666 0 0 rpy=0 0 0
- joint link2_link3: origin xyz=0.976531988691246 0 0 rpy=0 0 0 -> xyz=0.5584553558758178 0 0 rpy=0 0 0
- joint link3_link4: origin xyz=1.2517540676601264 0 0 rpy=0 0 0 -> xyz=2.1055454153171325 0 0 rpy=0 0 0
- joint link4_link5: origin xyz=2.4295077829422462 0 0 rpy=0 0 0 -> xyz=1.093697705160728 0 0 rpy=0 0 0
- joint link5_link6: origin xyz=1.5520066356970015 0 0 rpy=0 0 0 -> xyz=1.3719094999863397 0 0 rpy=0 0 0
- joint link6_link7: origin xyz=1.6191688742315353 0 0 rpy=0 0 0 -> xyz=1.2043036478969262 0 0 rpy=0 0 0

Commit message: ass6: tried making snakeLinks and snakeJoints dictionaries in order to add sensors to correct links... not working yet

File: body.urdf (robot description, URDF)
Before this commit: robot robot, 7 links, 6 joints
Links:
- added link link10, mass 2.744179784938587; collision box size=1.5759908568137497 0.5463651380497547 2.424454794319167; visual box size=1.5759908568137497 0.5463651380497547 2.424454794319167
- added link link8, mass 0.8896547422538897; collision box size=1.0476641458489055 1.4555388516660257 2.175649103398759; visual box size=1.0476641458489055 1.4555388516660257 2.175649103398759
- added link link9, mass 3.0213214817489584; collision box size=1.5759908568137497 1.9757121823453956 1.3984644717941375; visual box size=1.5759908568137497 1.9757121823453956 1.3984644717941375
- link link1: mass 3.798663505993619 -> 4.106872566472319; geometry collision box size=1.1370084449932207 1.776977119422215 1.8979868436234915; visual box size=1.1370084449932207 1.776977119422215 1.8979868436234915
- link link2: mass 0.1042664700510676 -> 2.775071715653663; geometry collision box size=1.4118138364622106 2.010955793127295 1.2262156645504265; visual box size=1.4118138364622106 2.010955793127295 1.2262156645504265
- link link3: mass 0.9388419124094066 -> 4.604978418214236; geometry collision box size=1.2424943250836156 1.6521199979142847 2.4274015788791434; visual box size=1.2424943250836156 1.6521199979142847 2.4274015788791434
- link link4: mass 0.2421340325638499 -> 0.6079835259703259; geometry collision box size=1.1797764769075885 1.4658315314210388 0.885417911056902; visual box size=1.1797764769075885 1.4658315314210388 0.885417911056902
- link link5: mass 2.1958066847564286 -> 4.350830326676799; geometry collision box size=1.3771974186973452 2.154697631654708 2.359107590602034; visual box size=1.3771974186973452 2.154697631654708 2.359107590602034
- link link6: mass 4.329982891495016 -> 2.059684380574808; geometry collision box size=2.4981099203475754 1.9735797470690954 0.8962240134615234; visual box size=2.4981099203475754 1.9735797470690954 0.8962240134615234
- link link7: mass 4.522658602844529 -> 4.853524763573348; geometry collision box size=1.4076731366445507 1.463111999008486 1.60364304770967; visual box size=1.4076731366445507 1.463111999008486 1.60364304770967
Joints:
- added joint link7_link8: type revolute, parent link7, child link8, origin xyz=1.4076731366445507 0 0 rpy=0 0 0, axis 0 1 0, limit lower=-3.14159 upper=3.14159 effort=0.0 velocity=0.0
- added joint link8_link9: type revolute, parent link8, child link9, origin xyz=1.0476641458489055 0 0 rpy=0 0 0, axis 0 1 0, limit lower=-3.14159 upper=3.14159 effort=0.0 velocity=0.0
- added joint link9_link10: type revolute, parent link9, child link10, origin xyz=1.5759908568137497 0 0 rpy=0 0 0, axis 0 1 0, limit lower=-3.14159 upper=3.14159 effort=0.0 velocity=0.0
- joint link1_link2: origin xyz=2.1681310979844666 0 0 rpy=0 0 0 -> xyz=1.1370084449932207 0 0 rpy=0 0 0
- joint link2_link3: origin xyz=0.5584553558758178 0 0 rpy=0 0 0 -> xyz=1.4118138364622106 0 0 rpy=0 0 0
- joint link3_link4: origin xyz=2.1055454153171325 0 0 rpy=0 0 0 -> xyz=1.2424943250836156 0 0 rpy=0 0 0
- joint link4_link5: origin xyz=1.093697705160728 0 0 rpy=0 0 0 -> xyz=1.1797764769075885 0 0 rpy=0 0 0
- joint link5_link6: origin xyz=1.3719094999863397 0 0 rpy=0 0 0 -> xyz=1.3771974186973452 0 0 rpy=0 0 0
- joint link6_link7: origin xyz=1.2043036478969262 0 0 rpy=0 0 0 -> xyz=2.4981099203475754 0 0 rpy=0 0 0

Commit message: ass6: still working through assigning sensor neurons to appropriate links

File: body.urdf (robot description, URDF)
Before this commit: robot robot, 10 links, 9 joints
Links:
- removed link link10
- removed link link9
- link link1: mass 4.106872566472319 -> 3.9827217711169247; geometry collision box size=2.480482197364479 1.546238724828834 1.7471366388772473; visual box size=2.480482197364479 1.546238724828834 1.7471366388772473
- link link2: mass 2.775071715653663 -> 1.4231030627284031; geometry collision box size=1.5287550541661405 1.3892062341850329 0.8458872123420884; visual box size=1.5287550541661405 1.3892062341850329 0.8458872123420884
- link link3: mass 4.604978418214236 -> 0.21214268213914422; geometry collision box size=1.1830497350944615 1.8214631775665986 1.1667967831755843; visual box size=1.1830497350944615 1.8214631775665986 1.1667967831755843
- link link4: mass 0.6079835259703259 -> 3.841650219171873; geometry collision box size=1.6773215758044302 0.7319319430486682 1.4578258166921434; visual box size=1.6773215758044302 0.7319319430486682 1.4578258166921434
- link link5: mass 4.350830326676799 -> 2.959809148669404; geometry collision box size=2.0973148686430747 1.436787657902716 1.4990529832392652; visual box size=2.0973148686430747 1.436787657902716 1.4990529832392652
- link link6: mass 2.059684380574808 -> 2.8098439176359347; geometry collision box size=1.6956479145621806 0.6681695716716749 1.9842321586406029; visual box size=1.6956479145621806 0.6681695716716749 1.9842321586406029
- link link7: mass 4.853524763573348 -> 2.165015299481659; geometry collision box size=1.839672165413739 1.7404081688742785 1.7654005992101984; visual box size=1.839672165413739 1.7404081688742785 1.7654005992101984
- link link8: mass 0.8896547422538897 -> 2.282844774048807; geometry collision box size=1.839672165413739 1.8034821462811303 1.9398527363323463; visual box size=1.839672165413739 1.8034821462811303 1.9398527363323463
Joints:
- removed joint link8_link9
- removed joint link9_link10
- joint link1_link2: origin xyz=1.1370084449932207 0 0 rpy=0 0 0 -> xyz=2.480482197364479 0 0 rpy=0 0 0
- joint link2_link3: origin xyz=1.4118138364622106 0 0 rpy=0 0 0 -> xyz=1.5287550541661405 0 0 rpy=0 0 0
- joint link3_link4: origin xyz=1.2424943250836156 0 0 rpy=0 0 0 -> xyz=1.1830497350944615 0 0 rpy=0 0 0
- joint link4_link5: origin xyz=1.1797764769075885 0 0 rpy=0 0 0 -> xyz=1.6773215758044302 0 0 rpy=0 0 0
- joint link5_link6: origin xyz=1.3771974186973452 0 0 rpy=0 0 0 -> xyz=2.0973148686430747 0 0 rpy=0 0 0
- joint link6_link7: origin xyz=2.4981099203475754 0 0 rpy=0 0 0 -> xyz=1.6956479145621806 0 0 rpy=0 0 0
- joint link7_link8: origin xyz=1.4076731366445507 0 0 rpy=0 0 0 -> xyz=1.839672165413739 0 0 rpy=0 0 0

Commit message: ass6: putting all cubes and joints inside the for loop

File: body.urdf (robot description, URDF)
Before this commit: robot robot, 8 links, 7 joints
Links:
- link link1: mass 3.9827217711169247 -> 3.834001950915705; geometry collision box size=0.8280566655434887 1.0824918666589702 0.8154832465038813; visual box size=0.8280566655434887 1.0824918666589702 0.8154832465038813
- link link2: mass 1.4231030627284031 -> 0.8113280056470379; geometry collision box size=1.1034673935454582 0.921582004658899 1.8504051716667804; visual box size=1.1034673935454582 0.921582004658899 1.8504051716667804
- link link3: mass 0.21214268213914422 -> 2.0918024165045583; geometry collision box size=1.2770572122858277 2.203612656763813 0.7993693987441004; visual box size=1.2770572122858277 2.203612656763813 0.7993693987441004
- link link4: mass 3.841650219171873 -> 3.045097763723798; geometry collision box size=1.3082331899602646 0.6559019369444035 1.6738640328913506; visual box size=1.3082331899602646 0.6559019369444035 1.6738640328913506
- link link5: mass 2.959809148669404 -> 1.1583454510565006; geometry collision box size=1.5410821489740287 2.003828726757831 0.8592837567030074; visual box size=1.5410821489740287 2.003828726757831 0.8592837567030074
- link link6: mass 2.8098439176359347 -> 1.949075235333424; geometry collision box size=2.1294968441232407 1.9008607688962158 2.3088360035419746; visual box size=2.1294968441232407 1.9008607688962158 2.3088360035419746
- link link7: mass 2.165015299481659 -> 2.3398774374935516; geometry collision box size=1.8815287768032196 1.7037625597494759 1.3408030599668004; visual box size=1.8815287768032196 1.7037625597494759 1.3408030599668004
- link link8: mass 2.282844774048807 -> 1.4290341288368547; geometry collision box size=0.7231110649992825 0.5860795465305457 0.6203456296881704; visual box size=0.7231110649992825 0.5860795465305457 0.6203456296881704
Joints:
- added joint link8_link9: type revolute, parent link8, child link9, origin xyz=0.7231110649992825 0 0 rpy=0 0 0, axis 0 1 0, limit lower=-3.14159 upper=3.14159 effort=0.0 velocity=0.0
- joint link1_link2: origin xyz=2.480482197364479 0 0 rpy=0 0 0 -> xyz=0.8280566655434887 0 0 rpy=0 0 0
- joint link2_link3: origin xyz=1.5287550541661405 0 0 rpy=0 0 0 -> xyz=1.1034673935454582 0 0 rpy=0 0 0
- joint link3_link4: origin xyz=1.1830497350944615 0 0 rpy=0 0 0 -> xyz=1.2770572122858277 0 0 rpy=0 0 0
- joint link4_link5: origin xyz=1.6773215758044302 0 0 rpy=0 0 0 -> xyz=1.3082331899602646 0 0 rpy=0 0 0
- joint link5_link6: origin xyz=2.0973148686430747 0 0 rpy=0 0 0 -> xyz=1.5410821489740287 0 0 rpy=0 0 0
- joint link6_link7: origin xyz=1.6956479145621806 0 0 rpy=0 0 0 -> xyz=2.1294968441232407 0 0 rpy=0 0 0
- joint link7_link8: origin xyz=1.839672165413739 0 0 rpy=0 0 0 -> xyz=1.8815287768032196 0 0 rpy=0 0 0
