Commit message: ass6: got all my links and joints inside for loop

File: body.urdf (robot description, URDF)
Before this commit: robot robot, 8 links, 8 joints
Links:
- removed link link8
- link link1: mass 3.834001950915705 -> 1.1066145838429764; geometry collision box size=2.129367276199608 2.088037232082881 1.9582234681446633; visual box size=2.129367276199608 2.088037232082881 1.9582234681446633
- link link2: mass 0.8113280056470379 -> 1.5874464276673876; geometry collision box size=0.7703720632472211 2.0865618379977557 1.4623603420823674; visual box size=0.7703720632472211 2.0865618379977557 1.4623603420823674
- link link3: mass 2.0918024165045583 -> 3.4384706096451048; geometry collision box size=0.6724455460591079 0.9452722422144229 1.604622215364843; visual box size=0.6724455460591079 0.9452722422144229 1.604622215364843
- link link4: mass 3.045097763723798 -> 3.379454320711373; geometry collision box size=2.1232916476533115 2.3213073394498274 1.3102645598199; visual box size=2.1232916476533115 2.3213073394498274 1.3102645598199
- link link5: mass 1.1583454510565006 -> 3.284394549170717; geometry collision box size=1.861451894137167 2.385297283738373 0.5249716531805351; visual box size=1.861451894137167 2.385297283738373 0.5249716531805351
- link link6: mass 1.949075235333424 -> 4.817904890204887; geometry collision box size=1.274463867987454 1.8184467991062343 1.9152053655869616; visual box size=1.274463867987454 1.8184467991062343 1.9152053655869616
- link link7: mass 2.3398774374935516 -> 4.393011656058708; geometry collision box size=1.998513991302332 0.5461922823005811 0.9489197836985275; visual box size=1.998513991302332 0.5461922823005811 0.9489197836985275
Joints:
- removed joint link7_link8
- removed joint link8_link9
- joint link1_link2: origin xyz=0.8280566655434887 0 0 rpy=0 0 0 -> xyz=2.129367276199608 0 1.9582234681446633 rpy=0 0 0
- joint link2_link3: origin xyz=1.1034673935454582 0 0 rpy=0 0 0 -> xyz=0.7703720632472211 0 0 rpy=0 0 0
- joint link3_link4: origin xyz=1.2770572122858277 0 0 rpy=0 0 0 -> xyz=0.6724455460591079 0 0 rpy=0 0 0
- joint link4_link5: origin xyz=1.3082331899602646 0 0 rpy=0 0 0 -> xyz=2.1232916476533115 0 0 rpy=0 0 0
- joint link5_link6: origin xyz=1.5410821489740287 0 0 rpy=0 0 0 -> xyz=1.861451894137167 0 0 rpy=0 0 0
- joint link6_link7: origin xyz=2.1294968441232407 0 0 rpy=0 0 0 -> xyz=1.274463867987454 0 0 rpy=0 0 0

Commit message: ass6: messing around with dictionary in for loop

File: body.urdf (robot description, URDF)
Before this commit: robot robot, 7 links, 6 joints
Links:
- removed link link5
- removed link link6
- removed link link7
- link link1: mass 1.1066145838429764 -> 4.863793457475549; geometry collision box size=2.4552763960366493 2.0375200481468445 1.8410511145539028; visual box size=2.4552763960366493 2.0375200481468445 1.8410511145539028
- link link2: mass 1.5874464276673876 -> 3.015995844810187; geometry collision box size=0.8917720769543667 2.2725468041200916 2.134811279208327; visual box size=0.8917720769543667 2.2725468041200916 2.134811279208327
- link link3: mass 3.4384706096451048 -> 3.88371645495643; geometry collision box size=1.704754481336114 2.474500123554672 2.0792703821810825; visual box size=1.704754481336114 2.474500123554672 2.0792703821810825
- link link4: mass 3.379454320711373 -> 1.3300870029468115; geometry collision box size=1.5986866618122593 1.1127984524797996 1.372130940273541; visual box size=1.5986866618122593 1.1127984524797996 1.372130940273541
Joints:
- removed joint link4_link5
- removed joint link5_link6
- removed joint link6_link7
- joint link1_link2: origin xyz=2.129367276199608 0 1.9582234681446633 rpy=0 0 0 -> xyz=2.4552763960366493 0 1.8410511145539028 rpy=0 0 0
- joint link2_link3: origin xyz=0.7703720632472211 0 0 rpy=0 0 0 -> xyz=0.8917720769543667 0 0 rpy=0 0 0
- joint link3_link4: origin xyz=0.6724455460591079 0 0 rpy=0 0 0 -> xyz=1.704754481336114 0 0 rpy=0 0 0

Commit message: ass6: got the neurons and synapses to work

File: body.urdf (robot description, URDF)
Before this commit: robot robot, 4 links, 3 joints
Links:
- added link link5, mass 2.4289096210608543; collision box size=1.403640620654004 0.6842267182332853 0.7124451242524601; visual box size=1.403640620654004 0.6842267182332853 0.7124451242524601
- added link link6, mass 3.780281651321038; collision box size=1.1166108189379447 1.0845692780071359 2.4926336806608207; visual box size=1.1166108189379447 1.0845692780071359 2.4926336806608207
- added link link7, mass 1.4316379077280965; collision box size=1.9770208029384742 2.4386487546153703 0.5057968729813695; visual box size=1.9770208029384742 2.4386487546153703 0.5057968729813695
- added link link8, mass 4.244893652436772; collision box size=0.9654073487181123 2.164879251994452 1.4375571444078208; visual box size=0.9654073487181123 2.164879251994452 1.4375571444078208
- link link1: mass 4.863793457475549 -> 2.91157921425272; geometry collision box size=0.5836955186020703 2.0229644086828475 1.611651914353078; visual box size=0.5836955186020703 2.0229644086828475 1.611651914353078
- link link2: mass 3.015995844810187 -> 2.005358407821621; geometry collision box size=2.1307483914644467 1.0119856231218727 1.3873409612087435; visual box size=2.1307483914644467 1.0119856231218727 1.3873409612087435
- link link3: mass 3.88371645495643 -> 2.414997124625266; geometry collision box size=1.5746237648805779 1.7878352948008716 2.1006508765379857; visual box size=1.5746237648805779 1.7878352948008716 2.1006508765379857
- link link4: mass 1.3300870029468115 -> 2.0430814230709533; geometry collision box size=0.6213311646664146 1.5710168054598426 1.9943107512586256; visual box size=0.6213311646664146 1.5710168054598426 1.9943107512586256
Joints:
- added joint link4_link5: type revolute, parent link4, child link5, origin xyz=0.6213311646664146 0 0 rpy=0 0 0, axis 0 1 0, limit lower=-3.14159 upper=3.14159 effort=0.0 velocity=0.0
- added joint link5_link6: type revolute, parent link5, child link6, origin xyz=1.403640620654004 0 0 rpy=0 0 0, axis 0 1 0, limit lower=-3.14159 upper=3.14159 effort=0.0 velocity=0.0
- added joint link6_link7: type revolute, parent link6, child link7, origin xyz=1.1166108189379447 0 0 rpy=0 0 0, axis 0 1 0, limit lower=-3.14159 upper=3.14159 effort=0.0 velocity=0.0
- added joint link7_link8: type revolute, parent link7, child link8, origin xyz=1.9770208029384742 0 0 rpy=0 0 0, axis 0 1 0, limit lower=-3.14159 upper=3.14159 effort=0.0 velocity=0.0
- joint link1_link2: origin xyz=2.4552763960366493 0 1.8410511145539028 rpy=0 0 0 -> xyz=0.5836955186020703 0 1.611651914353078 rpy=0 0 0
- joint link2_link3: origin xyz=0.8917720769543667 0 0 rpy=0 0 0 -> xyz=2.1307483914644467 0 0 rpy=0 0 0
- joint link3_link4: origin xyz=1.704754481336114 0 0 rpy=0 0 0 -> xyz=1.5746237648805779 0 0 rpy=0 0 0

Commit message: ass6: doing the readme

File: body.urdf (robot description, URDF)
Before this commit: robot robot, 8 links, 7 joints
Links:
- removed link link7
- removed link link8
- link link1: mass 2.91157921425272 -> 0.5699423405894627; geometry collision box size=1.4786509626676054 1.0509533013587005 0.6484035048533929; visual box size=1.4786509626676054 1.0509533013587005 0.6484035048533929
- link link2: mass 2.005358407821621 -> 2.244009752290839; geometry collision box size=1.631696265289404 2.312794260699036 0.8162539468185428; visual box size=1.631696265289404 2.312794260699036 0.8162539468185428
- link link3: mass 2.414997124625266 -> 0.46211810565230105; geometry collision box size=2.3850001015485613 1.6786853225982648 1.1745492563219382; visual box size=2.3850001015485613 1.6786853225982648 1.1745492563219382
- link link4: mass 2.0430814230709533 -> 1.0135353838887422; geometry collision box size=1.857932848313663 1.1379923310990714 1.2393800389588627; visual box size=1.857932848313663 1.1379923310990714 1.2393800389588627
- link link5: mass 2.4289096210608543 -> 4.889355052639309; geometry collision box size=0.5551429885364514 1.4017479045777141 1.986750855800506; visual box size=0.5551429885364514 1.4017479045777141 1.986750855800506
- link link6: mass 3.780281651321038 -> 2.570989466311449; geometry collision box size=1.388729203677046 1.6405475542235246 0.9628944812759228; visual box size=1.388729203677046 1.6405475542235246 0.9628944812759228
Joints:
- removed joint link6_link7
- removed joint link7_link8
- joint link1_link2: axis 0 1 0 -> 0 0 1; origin xyz=0.5836955186020703 0 1.611651914353078 rpy=0 0 0 -> xyz=1.4786509626676054 0 0.6484035048533929 rpy=0 0 0
- joint link2_link3: axis 0 1 0 -> 0 0 1; origin xyz=2.1307483914644467 0 0 rpy=0 0 0 -> xyz=1.631696265289404 0 0 rpy=0 0 0
- joint link3_link4: axis 0 1 0 -> 0 0 1; origin xyz=1.5746237648805779 0 0 rpy=0 0 0 -> xyz=2.3850001015485613 0 0 rpy=0 0 0
- joint link4_link5: axis 0 1 0 -> 0 0 1; origin xyz=0.6213311646664146 0 0 rpy=0 0 0 -> xyz=1.857932848313663 0 0 rpy=0 0 0
- joint link5_link6: axis 0 1 0 -> 0 0 1; origin xyz=1.403640620654004 0 0 rpy=0 0 0 -> xyz=0.5551429885364514 0 0 rpy=0 0 0

Commit message: ass6: edited readme

File: body.urdf (robot description, URDF)
Before this commit: robot robot, 6 links, 5 joints
Links:
- removed link link6
- link link1: mass 0.5699423405894627 -> 3.6355908362784186; geometry collision box size=0.9174513321291906 1.6599805481907115 1.5523960143713076; visual box size=0.9174513321291906 1.6599805481907115 1.5523960143713076
- link link2: mass 2.244009752290839 -> 2.9217673868040936; geometry collision box size=1.1014623348652615 1.8556890065829899 1.9162702702713679; visual box size=1.1014623348652615 1.8556890065829899 1.9162702702713679
- link link3: mass 0.46211810565230105 -> 3.159860612965357; geometry collision box size=2.3165642625885345 0.9629919024797893 2.0512985399203076; visual box size=2.3165642625885345 0.9629919024797893 2.0512985399203076
- link link4: mass 1.0135353838887422 -> 0.06407120806805056; geometry collision box size=2.1627879250026787 2.4114437842699576 2.02796818918205; visual box size=2.1627879250026787 2.4114437842699576 2.02796818918205
- link link5: mass 4.889355052639309 -> 1.1245890930196856; geometry collision box size=2.1645479331867072 2.1620304648555777 1.7080884388884165; visual box size=2.1645479331867072 2.1620304648555777 1.7080884388884165
Joints:
- removed joint link5_link6
- joint link1_link2: origin xyz=1.4786509626676054 0 0.6484035048533929 rpy=0 0 0 -> xyz=0.9174513321291906 0 1.5523960143713076 rpy=0 0 0
- joint link2_link3: origin xyz=1.631696265289404 0 0 rpy=0 0 0 -> xyz=1.1014623348652615 0 0 rpy=0 0 0
- joint link3_link4: origin xyz=2.3850001015485613 0 0 rpy=0 0 0 -> xyz=2.3165642625885345 0 0 rpy=0 0 0
- joint link4_link5: origin xyz=1.857932848313663 0 0 rpy=0 0 0 -> xyz=2.1627879250026787 0 0 rpy=0 0 0

Commit message: ass6: added random snake jpg

File: body.urdf (robot description, URDF)
Before this commit: robot robot, 5 links, 4 joints
Links:
- removed link link5
- link link1: mass 3.6355908362784186 -> 1.5423794864957996; geometry collision box size=1.2415631920853587 2.3956212505253918 2.1489956363438445; visual box size=1.2415631920853587 2.3956212505253918 2.1489956363438445
- link link2: mass 2.9217673868040936 -> 4.970383719628497; geometry collision box size=1.300829239691603 1.7550474037644168 1.539554337202965; visual box size=1.300829239691603 1.7550474037644168 1.539554337202965
- link link3: mass 3.159860612965357 -> 2.523718376968817; geometry collision box size=1.6307804813367524 1.0166957947158788 1.7181869538334105; visual box size=1.6307804813367524 1.0166957947158788 1.7181869538334105
- link link4: mass 0.06407120806805056 -> 4.581224946877182; geometry collision box size=1.7672048129285824 1.2374422889396572 0.5792046993859503; visual box size=1.7672048129285824 1.2374422889396572 0.5792046993859503
Joints:
- removed joint link4_link5
- joint link1_link2: axis 0 0 1 -> 0 1 0; origin xyz=0.9174513321291906 0 1.5523960143713076 rpy=0 0 0 -> xyz=1.2415631920853587 0 2.1489956363438445 rpy=0 0 0
- joint link2_link3: axis 0 0 1 -> 0 1 0; origin xyz=1.1014623348652615 0 0 rpy=0 0 0 -> xyz=1.300829239691603 0 0 rpy=0 0 0
- joint link3_link4: axis 0 0 1 -> 0 1 0; origin xyz=2.3165642625885345 0 0 rpy=0 0 0 -> xyz=1.6307804813367524 0 0 rpy=0 0 0

Commit message: a7: trying to reincorporate fitness / parallel hillclimber

File: body.urdf (robot description, URDF)
Before this commit: robot robot, 4 links, 3 joints
Links:
- link link1: mass 1.5423794864957996 -> 2.177722086738973; geometry collision box size=0.5886826013372439 0.7137672993085826 1.6872394628824283; visual box size=0.5886826013372439 0.7137672993085826 1.6872394628824283
- link link2: mass 4.970383719628497 -> 1.8508972923901246; geometry collision box size=0.5389090918428783 1.0501827919943099 1.7796709749368869; visual box size=0.5389090918428783 1.0501827919943099 1.7796709749368869
- link link3: mass 2.523718376968817 -> 1.276770374382461; geometry collision box size=0.7276690138673785 2.167523832617442 2.1979198245575757; visual box size=0.7276690138673785 2.167523832617442 2.1979198245575757
- link link4: mass 4.581224946877182 -> 2.8231485176342517; geometry collision box size=1.842685401305704 1.9845928237759765 0.7857461201516429; visual box size=1.842685401305704 1.9845928237759765 0.7857461201516429
Joints:
- joint link1_link2: origin xyz=1.2415631920853587 0 2.1489956363438445 rpy=0 0 0 -> xyz=0.5886826013372439 0 1.6872394628824283 rpy=0 0 0
- joint link2_link3: origin xyz=1.300829239691603 0 0 rpy=0 0 0 -> xyz=0.5389090918428783 0 0 rpy=0 0 0
- joint link3_link4: origin xyz=1.6307804813367524 0 0 rpy=0 0 0 -> xyz=0.7276690138673785 0 0 rpy=0 0 0

Commit message: a7: couldn't figure out fitness, but starting on random multiple dimension robot

File: body.urdf (robot description, URDF)
Before this commit: robot robot, 4 links, 3 joints
Links:
- added link link5, mass 1; collision box size=0.922456783616876 1.9296320215031793 0.6710673379482506; visual box size=0.922456783616876 1.9296320215031793 0.6710673379482506
- added link link6, mass 1; collision box size=0.9509034609355409 1.6363628085996875 2.1947952577879613; visual box size=0.9509034609355409 1.6363628085996875 2.1947952577879613
- added link link7, mass 1; collision box size=1.4669897291079323 2.241481190130647 1.2293799398070908; visual box size=1.4669897291079323 2.241481190130647 1.2293799398070908
- added link link8, mass 1; collision box size=2.1364332798055727 0.6350295395337902 1.4211158353977427; visual box size=2.1364332798055727 0.6350295395337902 1.4211158353977427
- added link link9, mass 1; collision box size=0.7572879175330647 1.869697343390577 1.1403585079831824; visual box size=0.7572879175330647 1.869697343390577 1.1403585079831824
- link link1: mass 2.177722086738973 -> 1; geometry collision box size=2.4398201727500477 2.4981591018014866 0.6102264845210801; visual box size=2.4398201727500477 2.4981591018014866 0.6102264845210801
- link link2: mass 1.8508972923901246 -> 1; geometry collision box size=1.8635178469164633 2.0200317589020713 1.3244603154617427; visual box size=1.8635178469164633 2.0200317589020713 1.3244603154617427
- link link3: mass 1.276770374382461 -> 1; geometry collision box size=1.42700896997149 1.0374225659796639 1.3928459567580447; visual box size=1.42700896997149 1.0374225659796639 1.3928459567580447
- link link4: mass 2.8231485176342517 -> 1; geometry collision box size=0.9585750359460425 1.765410526038368 1.6979412196711217; visual box size=0.9585750359460425 1.765410526038368 1.6979412196711217
Joints:
- added joint link4_link5: type revolute, parent link4, child link5, origin xyz=0.9585750359460425 0 0 rpy=0 0 0, axis 0 1 0, limit lower=-3.14159 upper=3.14159 effort=0.0 velocity=0.0
- added joint link5_link6: type revolute, parent link5, child link6, origin xyz=0.922456783616876 0 0 rpy=0 0 0, axis 0 1 0, limit lower=-3.14159 upper=3.14159 effort=0.0 velocity=0.0
- added joint link6_link7: type revolute, parent link6, child link7, origin xyz=0.9509034609355409 0 0 rpy=0 0 0, axis 0 1 0, limit lower=-3.14159 upper=3.14159 effort=0.0 velocity=0.0
- added joint link7_link8: type revolute, parent link7, child link8, origin xyz=1.4669897291079323 0 0 rpy=0 0 0, axis 0 1 0, limit lower=-3.14159 upper=3.14159 effort=0.0 velocity=0.0
- added joint link8_link9: type revolute, parent link8, child link9, origin xyz=2.1364332798055727 0 0 rpy=0 0 0, axis 0 1 0, limit lower=-3.14159 upper=3.14159 effort=0.0 velocity=0.0
- joint link1_link2: origin xyz=0.5886826013372439 0 1.6872394628824283 rpy=0 0 0 -> xyz=2.4398201727500477 0 0.6102264845210801 rpy=0 0 0
- joint link2_link3: origin xyz=0.5389090918428783 0 0 rpy=0 0 0 -> xyz=1.8635178469164633 0 0 rpy=0 0 0
- joint link3_link4: origin xyz=0.7276690138673785 0 0 rpy=0 0 0 -> xyz=1.42700896997149 0 0 rpy=0 0 0

Commit message: a7: working on new randomized robot .. thinking about using different methods for each branch of robot.

File: body.urdf (robot description, URDF)
Before this commit: robot robot, 9 links, 8 joints
Links:
- removed link link3
- removed link link4
- removed link link5
- removed link link6
- removed link link7
- removed link link8
- removed link link9
- link link1: mass 1 -> 100; geometry collision box size=2 2 2; visual box size=2 2 2
- link link2: geometry collision box size=1 1.5 1; visual box size=1 1.5 1
Joints:
- removed joint link1_link2
- removed joint link2_link3
- removed joint link3_link4
- removed joint link4_link5
- removed joint link5_link6
- removed joint link6_link7
- removed joint link7_link8
- removed joint link8_link9
- added joint link1_link2_xy: type revolute, parent link1, child link2, origin xyz=0 1 1 rpy=0 0 0, axis 0 0 1, limit lower=-3.14159 upper=3.14159 effort=0.0 velocity=0.0

Commit message: a7: working on building my random robot

File: body.urdf (robot description, URDF)
Before this commit: robot robot, 2 links, 1 joints
Links:
- removed link link1
- removed link link2
- added link link0_plusY, mass 1; collision box size=0.6969685659420934 1.521574368578586 0.806034545694764; visual box size=0.6969685659420934 1.521574368578586 0.806034545694764
- added link link1_plusY, mass 1; collision box size=0.369456859023147 0.8322037313123902 0.32922725364536; visual box size=0.369456859023147 0.8322037313123902 0.32922725364536
- added link link2_plusY, mass 1; collision box size=0.45875843512601727 0.8312122812782642 0.4669233804472521; visual box size=0.45875843512601727 0.8312122812782642 0.4669233804472521
- added link link3_plusY, mass 1; collision box size=0.2729152522662425 1.0951816036936917 0.4936370861820996; visual box size=0.2729152522662425 1.0951816036936917 0.4936370861820996
- added link link4_plusY, mass 1; collision box size=0.27193140668242344 0.7716482553974046 0.36058078461964127; visual box size=0.27193140668242344 0.7716482553974046 0.36058078461964127
- added link link5_plusY, mass 1; collision box size=0.4637465533936297 0.3527125925696388 0.4545959485362012; visual box size=0.4637465533936297 0.3527125925696388 0.4545959485362012
- added link link6_plusY, mass 1; collision box size=0.4238547495601491 0.3478900945632135 0.250910070058899; visual box size=0.4238547495601491 0.3478900945632135 0.250910070058899
- added link link7_plusY, mass 1; collision box size=0.4161115535466651 0.5662969019991869 0.4220625382893714; visual box size=0.4161115535466651 0.5662969019991869 0.4220625382893714
- added link rootLink, mass 100; collision box size=2 2 2; visual box size=2 2 2
Joints:
- removed joint link1_link2_xy
- added joint link0_plusY_link1_plusY: type revolute, parent link0_plusY, child link1_plusY, origin xyz=0 0.8322037313123902 0 rpy=0 0 0, axis 0 0 1, limit lower=-3.14159 upper=3.14159 effort=0.0 velocity=0.0
- added joint link1_plusY_link2_plusY: type revolute, parent link1_plusY, child link2_plusY, origin xyz=0 0.8312122812782642 0 rpy=0 0 0, axis 0 0 1, limit lower=-3.14159 upper=3.14159 effort=0.0 velocity=0.0
- added joint link2_plusY_link3_plusY: type revolute, parent link2_plusY, child link3_plusY, origin xyz=0 1.0951816036936917 0 rpy=0 0 0, axis 0 0 1, limit lower=-3.14159 upper=3.14159 effort=0.0 velocity=0.0
- added joint link3_plusY_link4_plusY: type revolute, parent link3_plusY, child link4_plusY, origin xyz=0 0.7716482553974046 0 rpy=0 0 0, axis 0 0 1, limit lower=-3.14159 upper=3.14159 effort=0.0 velocity=0.0
- added joint link4_plusY_link5_plusY: type revolute, parent link4_plusY, child link5_plusY, origin xyz=0 0.3527125925696388 0 rpy=0 0 0, axis 0 0 1, limit lower=-3.14159 upper=3.14159 effort=0.0 velocity=0.0
- added joint link5_plusY_link6_plusY: type revolute, parent link5_plusY, child link6_plusY, origin xyz=0 0.3478900945632135 0 rpy=0 0 0, axis 0 0 1, limit lower=-3.14159 upper=3.14159 effort=0.0 velocity=0.0
- added joint link6_plusY_link7_plusY: type revolute, parent link6_plusY, child link7_plusY, origin xyz=0 0.5662969019991869 0 rpy=0 0 0, axis 0 0 1, limit lower=-3.14159 upper=3.14159 effort=0.0 velocity=0.0
- added joint rootLink_plusY_link0_plusY: type revolute, parent rootLink, child link0_plusY, origin xyz=0 1 1 rpy=0 0 0, axis 0 0 1, limit lower=-3.14159 upper=3.14159 effort=0.0 velocity=0.0
