Commit message: a7: working on robot

File: body.urdf (robot description, URDF)
Before this commit: robot robot, 9 links, 8 joints
Links:
- removed link link2_plusY
- removed link link3_plusY
- removed link link4_plusY
- removed link link5_plusY
- removed link link6_plusY
- removed link link7_plusY
- added link link0_negX, mass 1; collision box size=1.4670792961071026 0.7176144213391731 0.5526061070991726; visual box size=1.4670792961071026 0.7176144213391731 0.5526061070991726
- added link link0_negY, mass 1; collision box size=0.6100939103654945 1.8111624362258059 0.9492317231221834; visual box size=0.6100939103654945 1.8111624362258059 0.9492317231221834
- added link link1_negX, mass 1; collision box size=1.5242679996959974 0.5564181387388207 0.8364735005362587; visual box size=1.5242679996959974 0.5564181387388207 0.8364735005362587
- added link link1_negY, mass 1; collision box size=0.5107996470629976 1.9395996005465077 0.9265179231795451; visual box size=0.5107996470629976 1.9395996005465077 0.9265179231795451
- added link link2_negY, mass 1; collision box size=0.9337579048331226 2.299890073358241 0.8862871595721353; visual box size=0.9337579048331226 2.299890073358241 0.8862871595721353
- link link0_plusY: geometry collision box size=0.956910142993472 0.9749251811657749 0.9755687668375372; visual box size=0.956910142993472 0.9749251811657749 0.9755687668375372
- link link1_plusY: geometry collision box size=0.6554143128455144 2.3105687384189935 0.9558044663398821; visual box size=0.6554143128455144 2.3105687384189935 0.9558044663398821
Joints:
- removed joint link1_plusY_link2_plusY
- removed joint link2_plusY_link3_plusY
- removed joint link3_plusY_link4_plusY
- removed joint link4_plusY_link5_plusY
- removed joint link5_plusY_link6_plusY
- removed joint link6_plusY_link7_plusY
- added joint link0_negX_link1_negX: type revolute, parent link0_negX, child link1_negX, origin xyz=-1.4670792961071026 0 0 rpy=0 0 0, axis 0 0 1, limit lower=-3.14159 upper=3.14159 effort=0.0 velocity=0.0
- added joint link0_negY_link1_negY: type revolute, parent link0_negY, child link1_negY, origin xyz=0 -1.8111624362258059 0 rpy=0 0 0, axis 0 0 1, limit lower=-3.14159 upper=3.14159 effort=0.0 velocity=0.0
- added joint link1_negY_link2_negY: type revolute, parent link1_negY, child link2_negY, origin xyz=0 -1.9395996005465077 0 rpy=0 0 0, axis 0 0 1, limit lower=-3.14159 upper=3.14159 effort=0.0 velocity=0.0
- added joint rootLink_negX_link0_negX: type revolute, parent rootLink, child link0_negX, origin xyz=-1 0 1 rpy=0 0 0, axis 0 0 1, limit lower=-3.14159 upper=3.14159 effort=0.0 velocity=0.0
- added joint rootLink_negY_link0_negY: type revolute, parent rootLink, child link0_negY, origin xyz=0 -1 1 rpy=0 0 0, axis 0 0 1, limit lower=-3.14159 upper=3.14159 effort=0.0 velocity=0.0
- joint link0_plusY_link1_plusY: origin xyz=0 0.8322037313123902 0 rpy=0 0 0 -> xyz=0 0.9749251811657749 0 rpy=0 0 0

Commit message: a7: trying new robot called the crawler

File: body.urdf (robot description, URDF)
Before this commit: robot robot, 8 links, 7 joints
Links:
- removed link link0_negX
- removed link link1_negX
- added link link2_plusY, mass 1; collision box size=0.5 0.5 3.5; visual box size=0.5 0.5 3.5
- link link0_negY: geometry collision box size=0.5 0.5 1; visual box size=0.5 0.5 1
- link link0_plusY: geometry collision box size=0.5 0.5 1; visual box size=0.5 0.5 1
- link link1_negY: geometry collision box size=0.5 2 0.5; visual box size=0.5 2 0.5
- link link1_plusY: geometry collision box size=0.5 2 0.5; visual box size=0.5 2 0.5
- link link2_negY: geometry collision box size=0.5 0.5 3.5; visual box size=0.5 0.5 3.5
Joints:
- removed joint link0_negX_link1_negX
- removed joint rootLink_negX_link0_negX
- removed joint rootLink_negY_link0_negY
- removed joint rootLink_plusY_link0_plusY
- added joint link1_plusY_link2_plusY: type revolute, parent link1_plusY, child link2_plusY, origin xyz=0 2 0 rpy=0 0 0, axis 0 1 0, limit lower=-3.14159 upper=3.14159 effort=0.0 velocity=0.0
- added joint rootLink_link0_negY: type revolute, parent rootLink, child link0_negY, origin xyz=0 -1 2 rpy=0 0 0, axis 0 0 1, limit lower=-3.14159 upper=3.14159 effort=0.0 velocity=0.0
- added joint rootLink_link0_plusY: type revolute, parent rootLink, child link0_plusY, origin xyz=0 1 2 rpy=0 0 0, axis 0 0 1, limit lower=-3.14159 upper=3.14159 effort=0.0 velocity=0.0
- joint link0_negY_link1_negY: axis 0 0 1 -> 1 0 0; origin xyz=0 -1.8111624362258059 0 rpy=0 0 0 -> xyz=0 0 1 rpy=0 0 0
- joint link0_plusY_link1_plusY: axis 0 0 1 -> 1 0 0; origin xyz=0 0.9749251811657749 0 rpy=0 0 0 -> xyz=0 0 1 rpy=0 0 0
- joint link1_negY_link2_negY: axis 0 0 1 -> 0 1 0; origin xyz=0 -1.9395996005465077 0 rpy=0 0 0 -> xyz=0 -2 0 rpy=0 0 0

Commit message: a7: working through various robot designs

File: body.urdf (robot description, URDF)
Before this commit: robot robot, 7 links, 6 joints
Links:
- removed link link1_negY
- removed link link1_plusY
- removed link link2_negY
- removed link link2_plusY
- link link0_negY: geometry collision box size=0.5011574638719957 0.5428205813767382 0.7954351177784331; visual box size=0.5011574638719957 0.5428205813767382 0.7954351177784331
- link link0_plusY: geometry collision box size=0.5011574638719957 0.5428205813767382 0.7954351177784331; visual box size=0.5011574638719957 0.5428205813767382 0.7954351177784331
- link rootLink: mass 100 -> 1; geometry collision box size=0.6148443530250567 0.6148443530250567 0.6148443530250567; visual box size=0.6148443530250567 0.6148443530250567 0.6148443530250567
Joints:
- removed joint link0_negY_link1_negY
- removed joint link0_plusY_link1_plusY
- removed joint link1_negY_link2_negY
- removed joint link1_plusY_link2_plusY
- joint rootLink_link0_negY: origin xyz=0 -1 2 rpy=0 0 0 -> xyz=-0.17855840561877034 -0.30742217651252834 0.11274128321434532 rpy=0 0 0
- joint rootLink_link0_plusY: origin xyz=0 1 2 rpy=0 0 0 -> xyz=-0.17855840561877034 0.30742217651252834 0.11274128321434532 rpy=0 0 0

Commit message: a7: added a plus z for the multiple leg robot

File: body.urdf (robot description, URDF)
Before this commit: robot robot, 3 links, 2 joints
Links:
- removed link link0_negY
- removed link link0_plusY
- added link link0_negX, mass 1; collision box size=2.497817334826541 0.9290454222181423 2.166544110172418; visual box size=2.497817334826541 0.9290454222181423 2.166544110172418
- added link link1_negX, mass 1; collision box size=1.3351583623029852 1.110442521306529 1.3511209182001356; visual box size=1.3351583623029852 1.110442521306529 1.3511209182001356
- added link link2_negX, mass 1; collision box size=0.8518376673276751 2.1691117509717737 2.4704163654624143; visual box size=0.8518376673276751 2.1691117509717737 2.4704163654624143
- link rootLink: geometry collision box size=2 2 2; visual box size=2 2 2
Joints:
- removed joint rootLink_link0_negY
- removed joint rootLink_link0_plusY
- added joint link0_negX_link1_negX: type revolute, parent link0_negX, child link1_negX, origin xyz=-2.497817334826541 0 0 rpy=0 0 0, axis 0 1 0, limit lower=-3.14159 upper=3.14159 effort=0.0 velocity=0.0
- added joint link1_negX_link2_negX: type revolute, parent link1_negX, child link2_negX, origin xyz=-1.3351583623029852 0 0 rpy=0 0 0, axis 0 0 1, limit lower=-3.14159 upper=3.14159 effort=0.0 velocity=0.0
- added joint rootLink_link0_negX: type revolute, parent rootLink, child link0_negX, origin xyz=-1 0 1 rpy=0 0 0, axis 0 0 1, limit lower=-3.14159 upper=3.14159 effort=0.0 velocity=0.0

Commit message: a7: started adding neurons

File: body.urdf (robot description, URDF)
Before this commit: robot robot, 4 links, 3 joints
Links:
- removed link link0_negX
- removed link link1_negX
- removed link link2_negX
- added link link0_plusZ, mass 1; collision box size=0.55788786982556 0.8498551274033985 0.9507023750393924; visual box size=0.55788786982556 0.8498551274033985 0.9507023750393924
- added link link1_plusZ, mass 1; collision box size=0.8569410709365406 0.8687092836111454 0.9511176821072163; visual box size=0.8569410709365406 0.8687092836111454 0.9511176821072163
Joints:
- removed joint link0_negX_link1_negX
- removed joint link1_negX_link2_negX
- removed joint rootLink_link0_negX
- added joint link0_plusZ_link1_plusZ: type revolute, parent link0_plusZ, child link1_plusZ, origin xyz=0 0 0.9507023750393924 rpy=0 0 0, axis 0 1 0, limit lower=-3.14159 upper=3.14159 effort=0.0 velocity=0.0
- added joint rootLink_link0_plusZ: type revolute, parent rootLink, child link0_plusZ, origin xyz=0 0 2 rpy=0 0 0, axis 0 0 1, limit lower=-3.14159 upper=3.14159 effort=0.0 velocity=0.0

Commit message: a7: working on neurons

File: body.urdf (robot description, URDF)
Before this commit: robot robot, 3 links, 2 joints
Links:
- added link link0_negX, mass 1; collision box size=1.3323598777886922 0.958134917752647 0.9610942812349437; visual box size=1.3323598777886922 0.958134917752647 0.9610942812349437
- added link link0_negY, mass 1; collision box size=0.6906021188441063 0.9331987942612268 0.7110582877913587; visual box size=0.6906021188441063 0.9331987942612268 0.7110582877913587
- added link link0_plusY, mass 1; collision box size=0.8804812224562878 1.4444904871522333 0.6898076116618639; visual box size=0.8804812224562878 1.4444904871522333 0.6898076116618639
- added link link1_negX, mass 1; collision box size=1.9472780206791538 0.6481951963934673 0.8715733302112489; visual box size=1.9472780206791538 0.6481951963934673 0.8715733302112489
- added link link1_negY, mass 1; collision box size=0.7189437968252861 1.4916244827637013 0.6165422251287863; visual box size=0.7189437968252861 1.4916244827637013 0.6165422251287863
- added link link1_plusY, mass 1; collision box size=0.631105680852545 0.8530784093615121 0.5358126654284201; visual box size=0.631105680852545 0.8530784093615121 0.5358126654284201
- added link link2_negX, mass 1; collision box size=1.840611132828142 0.6516842554664588 0.7937903030717797; visual box size=1.840611132828142 0.6516842554664588 0.7937903030717797
- added link link2_plusY, mass 1; collision box size=0.8607700161703913 0.9575244425409053 0.9726353477769611; visual box size=0.8607700161703913 0.9575244425409053 0.9726353477769611
- added link link2_plusZ, mass 1; collision box size=0.5147874819834535 0.5217436451782638 1.906764177207672; visual box size=0.5147874819834535 0.5217436451782638 1.906764177207672
- link link0_plusZ: geometry collision box size=0.8987021237771514 0.7071569996503871 0.8460148031581018; visual box size=0.8987021237771514 0.7071569996503871 0.8460148031581018
- link link1_plusZ: geometry collision box size=0.7542132441249909 0.8892213075000729 1.5418768352262904; visual box size=0.7542132441249909 0.8892213075000729 1.5418768352262904
Joints:
- added joint link0_negX_link1_negX: type revolute, parent link0_negX, child link1_negX, origin xyz=-1.3323598777886922 0 0 rpy=0 0 0, axis 1 0 0, limit lower=-3.14159 upper=3.14159 effort=0.0 velocity=0.0
- added joint link0_negY_link1_negY: type revolute, parent link0_negY, child link1_negY, origin xyz=0 -0.9331987942612268 0 rpy=0 0 0, axis 0 0 1, limit lower=-3.14159 upper=3.14159 effort=0.0 velocity=0.0
- added joint link0_plusY_link1_plusY: type revolute, parent link0_plusY, child link1_plusY, origin xyz=0 1.4444904871522333 0 rpy=0 0 0, axis 1 0 0, limit lower=-3.14159 upper=3.14159 effort=0.0 velocity=0.0
- added joint link1_negX_link2_negX: type revolute, parent link1_negX, child link2_negX, origin xyz=-1.9472780206791538 0 0 rpy=0 0 0, axis 0 0 1, limit lower=-3.14159 upper=3.14159 effort=0.0 velocity=0.0
- added joint link1_plusY_link2_plusY: type revolute, parent link1_plusY, child link2_plusY, origin xyz=0 0.8530784093615121 0 rpy=0 0 0, axis 0 0 1, limit lower=-3.14159 upper=3.14159 effort=0.0 velocity=0.0
- added joint link1_plusZ_link2_plusZ: type revolute, parent link1_plusZ, child link2_plusZ, origin xyz=0 0 1.5418768352262904 rpy=0 0 0, axis 0 1 0, limit lower=-3.14159 upper=3.14159 effort=0.0 velocity=0.0
- added joint rootLink_link0_negX: type revolute, parent rootLink, child link0_negX, origin xyz=-1 0 1 rpy=0 0 0, axis 0 1 0, limit lower=-3.14159 upper=3.14159 effort=0.0 velocity=0.0
- added joint rootLink_link0_negY: type revolute, parent rootLink, child link0_negY, origin xyz=0 -1 1 rpy=0 0 0, axis 0 0 1, limit lower=-3.14159 upper=3.14159 effort=0.0 velocity=0.0
- added joint rootLink_link0_plusY: type revolute, parent rootLink, child link0_plusY, origin xyz=0 1 1 rpy=0 0 0, axis 1 0 0, limit lower=-3.14159 upper=3.14159 effort=0.0 velocity=0.0
- joint link0_plusZ_link1_plusZ: axis 0 1 0 -> 1 0 0; origin xyz=0 0 0.9507023750393924 rpy=0 0 0 -> xyz=0 0 0.8460148031581018 rpy=0 0 0
- joint rootLink_link0_plusZ: axis 0 0 1 -> 1 0 0

Commit message: a7: fixed link names and joint names and solved my issue with sensor neurons

File: body.urdf (robot description, URDF)
Before this commit: robot robot, 12 links, 11 joints
Links:
- removed link link0_negX
- removed link link0_negY
- removed link link0_plusY
- removed link link0_plusZ
- removed link link1_negX
- removed link link1_negY
- removed link link1_plusY
- removed link link1_plusZ
- removed link link2_negX
- removed link link2_plusY
- removed link link2_plusZ
- added link link0negY, mass 1; collision box size=0.6046148970960536 0.8164554794041825 1.4269989418467117; visual box size=0.6046148970960536 0.8164554794041825 1.4269989418467117
- added link link0plusY, mass 1; collision box size=0.841871609125076 1.9854809677515706 1.3578816801115128; visual box size=0.841871609125076 1.9854809677515706 1.3578816801115128
- added link link1negY, mass 1; collision box size=0.5687464726391109 0.7727232309371068 1.0038200619908764; visual box size=0.5687464726391109 0.7727232309371068 1.0038200619908764
- added link link1plusY, mass 1; collision box size=0.50225260535696 0.7568994040373173 0.9169720758507719; visual box size=0.50225260535696 0.7568994040373173 0.9169720758507719
- added link link2negY, mass 1; collision box size=0.9119942846732448 0.7267530168656295 0.5856146078737622; visual box size=0.9119942846732448 0.7267530168656295 0.5856146078737622
- added link link2plusY, mass 1; collision box size=0.583647002126018 1.4224590260263275 1.0559815935040813; visual box size=0.583647002126018 1.4224590260263275 1.0559815935040813
Joints:
- removed joint link0_negX_link1_negX
- removed joint link0_negY_link1_negY
- removed joint link0_plusY_link1_plusY
- removed joint link0_plusZ_link1_plusZ
- removed joint link1_negX_link2_negX
- removed joint link1_plusY_link2_plusY
- removed joint link1_plusZ_link2_plusZ
- removed joint rootLink_link0_negX
- removed joint rootLink_link0_negY
- removed joint rootLink_link0_plusY
- removed joint rootLink_link0_plusZ
- added joint link0negY_link1negY: type revolute, parent link0negY, child link1negY, origin xyz=0 -0.8164554794041825 0 rpy=0 0 0, axis 0 1 0, limit lower=-3.14159 upper=3.14159 effort=0.0 velocity=0.0
- added joint link0plusY_link1plusY: type revolute, parent link0plusY, child link1plusY, origin xyz=0 1.9854809677515706 0 rpy=0 0 0, axis 0 0 1, limit lower=-3.14159 upper=3.14159 effort=0.0 velocity=0.0
- added joint link1negY_link2negY: type revolute, parent link1negY, child link2negY, origin xyz=0 -0.7727232309371068 0 rpy=0 0 0, axis 1 0 0, limit lower=-3.14159 upper=3.14159 effort=0.0 velocity=0.0
- added joint link1plusY_link2plusY: type revolute, parent link1plusY, child link2plusY, origin xyz=0 0.7568994040373173 0 rpy=0 0 0, axis 0 0 1, limit lower=-3.14159 upper=3.14159 effort=0.0 velocity=0.0
- added joint rootLink_link0negY: type revolute, parent rootLink, child link0negY, origin xyz=0 -1 2 rpy=0 0 0, axis 0 1 0, limit lower=-3.14159 upper=3.14159 effort=0.0 velocity=0.0
- added joint rootLink_link0plusY: type revolute, parent rootLink, child link0plusY, origin xyz=0 1 2 rpy=0 0 0, axis 1 0 0, limit lower=-3.14159 upper=3.14159 effort=0.0 velocity=0.0

Commit message: a7: edited readme

File: body.urdf (robot description, URDF)
Before this commit: robot robot, 7 links, 6 joints
Links:
- removed link link0negY
- removed link link0plusY
- removed link link1negY
- removed link link1plusY
- removed link link2negY
- removed link link2plusY
- added link link0_negY, mass 1; collision box size=0.5 0.5 1; visual box size=0.5 0.5 1
- added link link0_plusY, mass 1; collision box size=0.5 0.5 1; visual box size=0.5 0.5 1
- added link link1_negY, mass 1; collision box size=0.5 2 0.5; visual box size=0.5 2 0.5
- added link link1_plusY, mass 1; collision box size=0.5 2 0.5; visual box size=0.5 2 0.5
- added link link2_negY, mass 1; collision box size=0.5 0.5 3; visual box size=0.5 0.5 3
- added link link2_plusY, mass 1; collision box size=0.5 0.5 3; visual box size=0.5 0.5 3
- link rootLink: mass 1 -> 100
Joints:
- removed joint link0negY_link1negY
- removed joint link0plusY_link1plusY
- removed joint link1negY_link2negY
- removed joint link1plusY_link2plusY
- removed joint rootLink_link0negY
- removed joint rootLink_link0plusY
- added joint link0_negY_link1_negY: type revolute, parent link0_negY, child link1_negY, origin xyz=0 0 1 rpy=0 0 0, axis 1 0 0, limit lower=-3.14159 upper=3.14159 effort=0.0 velocity=0.0
- added joint link0_plusY_link1_plusY: type revolute, parent link0_plusY, child link1_plusY, origin xyz=0 0 1 rpy=0 0 0, axis 1 0 0, limit lower=-3.14159 upper=3.14159 effort=0.0 velocity=0.0
- added joint link1_negY_link2_negY: type revolute, parent link1_negY, child link2_negY, origin xyz=0 -2 0 rpy=0 0 0, axis 0 1 0, limit lower=-3.14159 upper=3.14159 effort=0.0 velocity=0.0
- added joint link1_plusY_link2_plusY: type revolute, parent link1_plusY, child link2_plusY, origin xyz=0 2 0 rpy=0 0 0, axis 0 1 0, limit lower=-3.14159 upper=3.14159 effort=0.0 velocity=0.0
- added joint rootLink_link0_negY: type revolute, parent rootLink, child link0_negY, origin xyz=0 -1 2 rpy=0 0 0, axis 0 0 1, limit lower=-3.14159 upper=3.14159 effort=0.0 velocity=0.0
- added joint rootLink_link0_plusY: type revolute, parent rootLink, child link0_plusY, origin xyz=0 1 2 rpy=0 0 0, axis 0 0 1, limit lower=-3.14159 upper=3.14159 effort=0.0 velocity=0.0

Commit message: a7: added one layer of hidden neurons

File: body.urdf (robot description, URDF)
Before this commit: robot robot, 7 links, 6 joints
Links:
- removed link link0_negY
- removed link link0_plusY
- removed link link1_negY
- removed link link1_plusY
- removed link link2_negY
- removed link link2_plusY
- added link link0negX, mass 1; collision box size=1.3323598777886922 1.416269835505294 1.4221885624698873; visual box size=1.3323598777886922 1.416269835505294 1.4221885624698873
- added link link0negY, mass 1; collision box size=0.8812042376882124 0.9331987942612268 0.9221165755827173; visual box size=0.8812042376882124 0.9331987942612268 0.9221165755827173
- added link link0plusY, mass 1; collision box size=1.2609624449125756 1.4444904871522333 0.8796152233237278; visual box size=1.2609624449125756 1.4444904871522333 0.8796152233237278
- added link link0plusZ, mass 1; collision box size=1.2974042475543028 0.9143139993007743 0.8460148031581018; visual box size=1.2974042475543028 0.9143139993007743 0.8460148031581018
- added link link1negX, mass 1; collision box size=1.9472780206791538 0.7963903927869346 1.2431466604224979; visual box size=1.9472780206791538 0.7963903927869346 1.2431466604224979
- added link link1negY, mass 1; collision box size=0.9378875936505721 1.4916244827637013 0.7330844502575726; visual box size=0.9378875936505721 1.4916244827637013 0.7330844502575726
- added link link1plusY, mass 1; collision box size=0.9288780283717567 0.8530784093615121 0.7382919975235068; visual box size=0.9288780283717567 0.8530784093615121 0.7382919975235068
- added link link1plusZ, mass 1; collision box size=1.0084264882499818 1.2784426150001458 1.5418768352262904; visual box size=1.0084264882499818 1.2784426150001458 1.5418768352262904
- added link link2negX, mass 1; collision box size=1.840611132828142 0.8033685109329176 1.0875806061435593; visual box size=1.840611132828142 0.8033685109329176 1.0875806061435593
- added link link2plusY, mass 1; collision box size=1.2215400323407826 0.9575244425409053 1.4452706955539223; visual box size=1.2215400323407826 0.9575244425409053 1.4452706955539223
- added link link2plusZ, mass 1; collision box size=0.5295749639669071 0.5434872903565274 1.906764177207672; visual box size=0.5295749639669071 0.5434872903565274 1.906764177207672
- link rootLink: mass 100 -> 5
Joints:
- removed joint link0_negY_link1_negY
- removed joint link0_plusY_link1_plusY
- removed joint link1_negY_link2_negY
- removed joint link1_plusY_link2_plusY
- removed joint rootLink_link0_negY
- removed joint rootLink_link0_plusY
- added joint link0negX_link1negX: type revolute, parent link0negX, child link1negX, origin xyz=-1.3323598777886922 0 0 rpy=0 0 0, axis 1 0 0, limit lower=-3.14159 upper=3.14159 effort=0.0 velocity=0.0
- added joint link0negY_link1negY: type revolute, parent link0negY, child link1negY, origin xyz=0 -0.9331987942612268 0 rpy=0 0 0, axis 0 0 1, limit lower=-3.14159 upper=3.14159 effort=0.0 velocity=0.0
- added joint link0plusY_link1plusY: type revolute, parent link0plusY, child link1plusY, origin xyz=0 1.4444904871522333 0 rpy=0 0 0, axis 1 0 0, limit lower=-3.14159 upper=3.14159 effort=0.0 velocity=0.0
- added joint link0plusZ_link1plusZ: type revolute, parent link0plusZ, child link1plusZ, origin xyz=0 0 0.8460148031581018 rpy=0 0 0, axis 1 0 0, limit lower=-3.14159 upper=3.14159 effort=0.0 velocity=0.0
- added joint link1negX_link2negX: type revolute, parent link1negX, child link2negX, origin xyz=-1.9472780206791538 0 0 rpy=0 0 0, axis 0 0 1, limit lower=-3.14159 upper=3.14159 effort=0.0 velocity=0.0
- added joint link1plusY_link2plusY: type revolute, parent link1plusY, child link2plusY, origin xyz=0 0.8530784093615121 0 rpy=0 0 0, axis 0 0 1, limit lower=-3.14159 upper=3.14159 effort=0.0 velocity=0.0
- added joint link1plusZ_link2plusZ: type revolute, parent link1plusZ, child link2plusZ, origin xyz=0 0 1.5418768352262904 rpy=0 0 0, axis 0 1 0, limit lower=-3.14159 upper=3.14159 effort=0.0 velocity=0.0
- added joint rootLink_link0negX: type revolute, parent rootLink, child link0negX, origin xyz=-1 0 1 rpy=0 0 0, axis 0 1 0, limit lower=-3.14159 upper=3.14159 effort=0.0 velocity=0.0
- added joint rootLink_link0negY: type revolute, parent rootLink, child link0negY, origin xyz=0 -1 1 rpy=0 0 0, axis 0 0 1, limit lower=-3.14159 upper=3.14159 effort=0.0 velocity=0.0
- added joint rootLink_link0plusY: type revolute, parent rootLink, child link0plusY, origin xyz=0 1 1 rpy=0 0 0, axis 1 0 0, limit lower=-3.14159 upper=3.14159 effort=0.0 velocity=0.0
- added joint rootLink_link0plusZ: type revolute, parent rootLink, child link0plusZ, origin xyz=0 0 2 rpy=0 0 0, axis 1 0 0, limit lower=-3.14159 upper=3.14159 effort=0.0 velocity=0.0
