Commit message: a7: trying a new robot generation method using lists called New_PlusY

File: body.urdf (robot description, URDF)
Before this commit: robot robot, 12 links, 11 joints
Links:
- removed link link0negX
- removed link link0negY
- removed link link0plusY
- removed link link0plusZ
- removed link link1negX
- removed link link1negY
- removed link link1plusY
- removed link link1plusZ
- removed link link2negX
- removed link link2plusY
- removed link link2plusZ
- removed link rootLink
- added link link0, mass 1; collision box size=1.3941171454887158 1.3941171454887158 1.3941171454887158; visual box size=1.3941171454887158 1.3941171454887158 1.3941171454887158
- added link link1, mass 1; collision box size=0.8858908890997076 0.8858908890997076 0.8858908890997076; visual box size=0.8858908890997076 0.8858908890997076 0.8858908890997076
- added link link2, mass 1; collision box size=0.9863747260399148 0.9863747260399148 0.9863747260399148; visual box size=0.9863747260399148 0.9863747260399148 0.9863747260399148
Joints:
- removed joint link0negX_link1negX
- removed joint link0negY_link1negY
- removed joint link0plusY_link1plusY
- removed joint link0plusZ_link1plusZ
- removed joint link1negX_link2negX
- removed joint link1plusY_link2plusY
- removed joint link1plusZ_link2plusZ
- removed joint rootLink_link0negX
- removed joint rootLink_link0negY
- removed joint rootLink_link0plusY
- removed joint rootLink_link0plusZ
- added joint link0_link1: type revolute, parent link0, child link1, origin xyz=1.3359902587578123 0.8076597987913037 1.290835739921795 rpy=0 0 0, axis 1 0 0, limit lower=-3.14159 upper=3.14159 effort=0.0 velocity=0.0
- added joint link1_link2: type revolute, parent link1, child link2, origin xyz=1.280147525411262 0.6154359999497544 0.6579466700042922 rpy=0 0 0, axis 1 0 0, limit lower=-3.14159 upper=3.14159 effort=0.0 velocity=0.0

Commit message: a7: oof.. trying to figure out 3d generation

File: body.urdf (robot description, URDF)
Before this commit: robot robot, 3 links, 2 joints
Links:
- added link rootLink, mass 1; collision box size=2 2 2; visual box size=2 2 2
- link link0: geometry collision box size=1 1 1; visual box size=1 1 1
- link link1: geometry collision box size=1 1 1; visual box size=1 1 1
- link link2: geometry collision box size=1 1 1; visual box size=1 1 1
Joints:
- added joint rootLink_link0: type revolute, parent rootLink, child link0, origin xyz=0 1.0 2 rpy=0 0 0, axis 0 1 0, limit lower=-3.14159 upper=3.14159 effort=0.0 velocity=0.0
- joint link0_link1: axis 1 0 0 -> 0 1 0; origin xyz=1.3359902587578123 0.8076597987913037 1.290835739921795 rpy=0 0 0 -> xyz=0 1 0 rpy=0 0 0
- joint link1_link2: origin xyz=1.280147525411262 0.6154359999497544 0.6579466700042922 rpy=0 0 0 -> xyz=0 1 0 rpy=0 0 0

Commit message: a7: getting closer

File: body.urdf (robot description, URDF)
Before this commit: robot robot, 4 links, 3 joints
Links:
- removed link link0
- added link link3, mass 1; collision box size=1 1 1; visual box size=1 1 1
- added link link4, mass 1; collision box size=1 1 1; visual box size=1 1 1
- added link link5, mass 1; collision box size=1 1 1; visual box size=1 1 1
- added link link6, mass 1; collision box size=1 1 1; visual box size=1 1 1
- added link link7, mass 1; collision box size=1 1 1; visual box size=1 1 1
- added link link8, mass 1; collision box size=1 1 1; visual box size=1 1 1
- added link link9, mass 1; collision box size=1 1 1; visual box size=1 1 1
- link rootLink: geometry collision box size=1 1 1; visual box size=1 1 1
Joints:
- removed joint link0_link1
- removed joint rootLink_link0
- added joint link2_link3: type revolute, parent link2, child link3, origin xyz=0.5 0.5 0 rpy=0 0 0, axis 1 0 0, limit lower=-3.14159 upper=3.14159 effort=0.0 velocity=0.0
- added joint link3_link4: type revolute, parent link3, child link4, origin xyz=0.5 0.5 0 rpy=0 0 0, axis 0 1 0, limit lower=-3.14159 upper=3.14159 effort=0.0 velocity=0.0
- added joint link4_link5: type revolute, parent link4, child link5, origin xyz=0.5 0 0.5 rpy=0 0 0, axis 1 0 0, limit lower=-3.14159 upper=3.14159 effort=0.0 velocity=0.0
- added joint link5_link6: type revolute, parent link5, child link6, origin xyz=0 0.5 0.5 rpy=0 0 0, axis 1 0 0, limit lower=-3.14159 upper=3.14159 effort=0.0 velocity=0.0
- added joint link6_link7: type revolute, parent link6, child link7, origin xyz=0.5 0.5 0 rpy=0 0 0, axis 0 0 1, limit lower=-3.14159 upper=3.14159 effort=0.0 velocity=0.0
- added joint link7_link8: type revolute, parent link7, child link8, origin xyz=0.5 0.5 0 rpy=0 0 0, axis 0 0 1, limit lower=-3.14159 upper=3.14159 effort=0.0 velocity=0.0
- added joint link8_link9: type revolute, parent link8, child link9, origin xyz=0 0.5 0.5 rpy=0 0 0, axis 0 1 0, limit lower=-3.14159 upper=3.14159 effort=0.0 velocity=0.0
- added joint rootLink_link1: type revolute, parent rootLink, child link1, origin xyz=0 0.5 3 rpy=0 0 0, axis 0 1 0, limit lower=-3.14159 upper=3.14159 effort=0.0 velocity=0.0
- joint link1_link2: axis 1 0 0 -> 0 1 0; origin xyz=0 1 0 rpy=0 0 0 -> xyz=0.5 0.5 0 rpy=0 0 0

Commit message: a7: still working through 3d robo generation

File: body.urdf (robot description, URDF)
Before this commit: robot robot, 10 links, 9 joints
Links:
- removed link link8
- removed link link9
- removed link rootLink
- added link link0, mass 100; collision box size=1 1 1; visual box size=1 1 1
Joints:
- removed joint link7_link8
- removed joint link8_link9
- removed joint rootLink_link1
- added joint link0_link1: type revolute, parent link0, child link1, origin xyz=0 0 1 rpy=0 0 0, axis 0 0 1, limit lower=-3.14159 upper=3.14159 effort=0.0 velocity=0.0
- joint link1_link2: axis 0 1 0 -> 0 0 1
- joint link2_link3: axis 1 0 0 -> 0 0 1
- joint link4_link5: origin xyz=0.5 0 0.5 rpy=0 0 0 -> xyz=0.5 0.5 0 rpy=0 0 0
- joint link5_link6: axis 1 0 0 -> 0 0 1; origin xyz=0 0.5 0.5 rpy=0 0 0 -> xyz=0.5 0 0.5 rpy=0 0 0
- joint link6_link7: axis 0 0 1 -> 1 0 0; origin xyz=0.5 0.5 0 rpy=0 0 0 -> xyz=0 0.5 0.5 rpy=0 0 0

Commit message: a7: got the joint positions and link positions in the right spot

File: body.urdf (robot description, URDF)
Before this commit: robot robot, 8 links, 7 joints
Links:
- removed link link6
- removed link link7
- link link0: mass 100 -> 1; geometry collision box size=0.31902781811705366 0.23817637164991387 0.59586076401173; visual box size=0.31902781811705366 0.23817637164991387 0.59586076401173
- link link1: geometry collision box size=0.31902781811705366 0.23817637164991387 0.59586076401173; visual box size=0.31902781811705366 0.23817637164991387 0.59586076401173
- link link2: geometry collision box size=0.9848244416424998 0.6772509897755892 0.3267883794753389; visual box size=0.9848244416424998 0.6772509897755892 0.3267883794753389
- link link3: geometry collision box size=0.6506140350167084 0.5638194275469663 0.9514693436715211; visual box size=0.6506140350167084 0.5638194275469663 0.9514693436715211
- link link4: geometry collision box size=0.7102208819219964 0.7020414126144296 0.9095591617326935; visual box size=0.7102208819219964 0.7020414126144296 0.9095591617326935
- link link5: geometry collision box size=0.5720359850583352 0.9936504624611684 0.3902019549213683; visual box size=0.5720359850583352 0.9936504624611684 0.3902019549213683
Joints:
- removed joint link5_link6
- removed joint link6_link7
- joint link0_link1: axis 0 0 1 -> 0 1 0; origin xyz=0 0 1 rpy=0 0 0 -> xyz=0 0 0.59586076401173 rpy=0 0 0
- joint link1_link2: origin xyz=0.5 0.5 0 rpy=0 0 0 -> xyz=0 0.11908818582495694 0.297930382005865 rpy=0 0 0
- joint link2_link3: origin xyz=0.5 0.5 0 rpy=0 0 0 -> xyz=0.4924122208212499 0.3386254948877946 0 rpy=0 0 0
- joint link3_link4: axis 0 1 0 -> 0 0 1; origin xyz=0.5 0.5 0 rpy=0 0 0 -> xyz=0.3253070175083542 0 0.47573467183576057 rpy=0 0 0
- joint link4_link5: origin xyz=0.5 0.5 0 rpy=0 0 0 -> xyz=0 0.3510207063072148 0.45477958086634673 rpy=0 0 0

Commit message: a7: working with a rootlink. going to add symmetrical arm next

File: body.urdf (robot description, URDF)
Before this commit: robot robot, 6 links, 5 joints
Links:
- removed link link0
- added link link6, mass 1; collision box size=0.6925594297625861 0.6510435399130685 0.4398390200652735; visual box size=0.6925594297625861 0.6510435399130685 0.4398390200652735
- added link link7, mass 1; collision box size=0.8080134057667185 0.7301788392709938 0.9196463290528545; visual box size=0.8080134057667185 0.7301788392709938 0.9196463290528545
- added link link8, mass 1; collision box size=0.2617642361186893 0.5997388584837322 0.7998028621963662; visual box size=0.2617642361186893 0.5997388584837322 0.7998028621963662
- added link rootLink, mass 100; collision box size=1 1 1; visual box size=1 1 1
- link link1: geometry collision box size=0 0 1; visual box size=0 0 1
- link link2: geometry collision box size=0.7980087389874271 0.7248477380873524 0.5229687150416005; visual box size=0.7980087389874271 0.7248477380873524 0.5229687150416005
- link link3: geometry collision box size=0.27594535799703596 0.3448645811831982 0.40396826714724443; visual box size=0.27594535799703596 0.3448645811831982 0.40396826714724443
- link link4: geometry collision box size=0.7537221015505091 0.8902956715524528 0.23743749226051758; visual box size=0.7537221015505091 0.8902956715524528 0.23743749226051758
- link link5: geometry collision box size=0.5049260132746789 0.6753848052468574 0.2804771672599361; visual box size=0.5049260132746789 0.6753848052468574 0.2804771672599361
Joints:
- removed joint link0_link1
- added joint link5_link6: type revolute, parent link5, child link6, origin xyz=-0.25246300663733945 0 0.14023858362996805 rpy=0 0 0, axis 0 0 1, limit lower=-3.14159 upper=3.14159 effort=0.0 velocity=0.0
- added joint link6_link7: type revolute, parent link6, child link7, origin xyz=-0.34627971488129305 0.32552176995653426 0 rpy=0 0 0, axis 0 1 0, limit lower=-3.14159 upper=3.14159 effort=0.0 velocity=0.0
- added joint link7_link8: type revolute, parent link7, child link8, origin xyz=-0.40400670288335927 0.3650894196354969 0 rpy=0 0 0, axis 0 1 0, limit lower=-3.14159 upper=3.14159 effort=0.0 velocity=0.0
- added joint rootLink_link1: type revolute, parent rootLink, child link1, origin xyz=0 0 1 rpy=0 0 0, axis 0 1 0, limit lower=-3.14159 upper=3.14159 effort=0.0 velocity=0.0
- joint link1_link2: axis 0 0 1 -> 1 0 0; origin xyz=0 0.11908818582495694 0.297930382005865 rpy=0 0 0 -> xyz=0 0.0 0.5 rpy=0 0 0
- joint link2_link3: origin xyz=0.4924122208212499 0.3386254948877946 0 rpy=0 0 0 -> xyz=-0.39900436949371354 0.3624238690436762 0 rpy=0 0 0
- joint link3_link4: axis 0 0 1 -> 1 0 0; origin xyz=0.3253070175083542 0 0.47573467183576057 rpy=0 0 0 -> xyz=-0.13797267899851798 0.1724322905915991 0 rpy=0 0 0
- joint link4_link5: origin xyz=0 0.3510207063072148 0.45477958086634673 rpy=0 0 0 -> xyz=0 0.4451478357762264 0.11871874613025879 rpy=0 0 0

Commit message: a7: completed the 3d symmetrical robot.. minor tweaks from here on out

File: body.urdf (robot description, URDF)
Before this commit: robot robot, 9 links, 8 joints
Links:
- removed link link1
- removed link link2
- removed link link3
- removed link link4
- removed link link5
- removed link link6
- removed link link7
- removed link link8
- added link link1NNP, mass 1; collision box size=0 0 1; visual box size=0 0 1
- added link link1NPP, mass 1; collision box size=0 0 1; visual box size=0 0 1
- added link link2NNP, mass 1; collision box size=0.7498478708294258 0.26101156603270914 0.8832383205505767; visual box size=0.7498478708294258 0.26101156603270914 0.8832383205505767
- added link link2NPP, mass 1; collision box size=0.7498478708294258 0.26101156603270914 0.8832383205505767; visual box size=0.7498478708294258 0.26101156603270914 0.8832383205505767
- added link link3NNP, mass 1; collision box size=0.9954560010364701 0.3964666000046848 0.5693563227615959; visual box size=0.9954560010364701 0.3964666000046848 0.5693563227615959
- added link link3NPP, mass 1; collision box size=0.9954560010364701 0.3964666000046848 0.5693563227615959; visual box size=0.9954560010364701 0.3964666000046848 0.5693563227615959
- added link link4NNP, mass 1; collision box size=0.6709729028664496 0.38532898916222746 0.6452670523584918; visual box size=0.6709729028664496 0.38532898916222746 0.6452670523584918
- added link link4NPP, mass 1; collision box size=0.6709729028664496 0.38532898916222746 0.6452670523584918; visual box size=0.6709729028664496 0.38532898916222746 0.6452670523584918
- added link link5NNP, mass 1; collision box size=0.7911881963811187 0.4613021044645003 0.25579979857095564; visual box size=0.7911881963811187 0.4613021044645003 0.25579979857095564
- added link link5NPP, mass 1; collision box size=0.7911881963811187 0.4613021044645003 0.25579979857095564; visual box size=0.7911881963811187 0.4613021044645003 0.25579979857095564
- added link link6NNP, mass 1; collision box size=0.6825399765579748 0.5811535194825307 0.4990919572185397; visual box size=0.6825399765579748 0.5811535194825307 0.4990919572185397
- added link link6NPP, mass 1; collision box size=0.6825399765579748 0.5811535194825307 0.4990919572185397; visual box size=0.6825399765579748 0.5811535194825307 0.4990919572185397
- added link link7NNP, mass 1; collision box size=0.6622487882592194 0.30833028953292446 0.6533074618987961; visual box size=0.6622487882592194 0.30833028953292446 0.6533074618987961
- added link link7NPP, mass 1; collision box size=0.6622487882592194 0.30833028953292446 0.6533074618987961; visual box size=0.6622487882592194 0.30833028953292446 0.6533074618987961
- link rootLink: mass 100 -> 10; geometry collision box size=0.4 0.4 0.4; visual box size=0.4 0.4 0.4
Joints:
- removed joint link1_link2
- removed joint link2_link3
- removed joint link3_link4
- removed joint link4_link5
- removed joint link5_link6
- removed joint link6_link7
- removed joint link7_link8
- removed joint rootLink_link1
- added joint link1NNP_link2NNP: type revolute, parent link1NNP, child link2NNP, origin xyz=0.0 0 0.5 rpy=0 0 0, axis 0 0 1, limit lower=-3.14159 upper=3.14159 effort=0.0 velocity=0.0
- added joint link1NPP_link2NPP: type revolute, parent link1NPP, child link2NPP, origin xyz=0.0 0 0.5 rpy=0 0 0, axis 0 0 1, limit lower=-3.14159 upper=3.14159 effort=0.0 velocity=0.0
- added joint link2NNP_link3NNP: type revolute, parent link2NNP, child link3NNP, origin xyz=-0.3749239354147129 0 0.44161916027528836 rpy=0 0 0, axis 0 0 1, limit lower=-3.14159 upper=3.14159 effort=0.0 velocity=0.0
- added joint link2NPP_link3NPP: type revolute, parent link2NPP, child link3NPP, origin xyz=-0.3749239354147129 0 0.44161916027528836 rpy=0 0 0, axis 0 0 1, limit lower=-3.14159 upper=3.14159 effort=0.0 velocity=0.0
- added joint link3NNP_link4NNP: type revolute, parent link3NNP, child link4NNP, origin xyz=-0.49772800051823507 0 0.28467816138079793 rpy=0 0 0, axis 0 1 0, limit lower=-3.14159 upper=3.14159 effort=0.0 velocity=0.0
- added joint link3NPP_link4NPP: type revolute, parent link3NPP, child link4NPP, origin xyz=-0.49772800051823507 0 0.28467816138079793 rpy=0 0 0, axis 0 1 0, limit lower=-3.14159 upper=3.14159 effort=0.0 velocity=0.0
- added joint link4NNP_link5NNP: type revolute, parent link4NNP, child link5NNP, origin xyz=-0.3354864514332248 -0.19266449458111373 0 rpy=0 0 0, axis 1 0 0, limit lower=-3.14159 upper=3.14159 effort=0.0 velocity=0.0
- added joint link4NPP_link5NPP: type revolute, parent link4NPP, child link5NPP, origin xyz=-0.3354864514332248 0.19266449458111373 0 rpy=0 0 0, axis 1 0 0, limit lower=-3.14159 upper=3.14159 effort=0.0 velocity=0.0
- added joint link5NNP_link6NNP: type revolute, parent link5NNP, child link6NNP, origin xyz=-0.39559409819055935 -0.23065105223225016 0 rpy=0 0 0, axis 0 0 1, limit lower=-3.14159 upper=3.14159 effort=0.0 velocity=0.0
- added joint link5NPP_link6NPP: type revolute, parent link5NPP, child link6NPP, origin xyz=-0.39559409819055935 0.23065105223225016 0 rpy=0 0 0, axis 0 0 1, limit lower=-3.14159 upper=3.14159 effort=0.0 velocity=0.0
- added joint link6NNP_link7NNP: type revolute, parent link6NNP, child link7NNP, origin xyz=-0.3412699882789874 0 0.24954597860926986 rpy=0 0 0, axis 1 0 0, limit lower=-3.14159 upper=3.14159 effort=0.0 velocity=0.0
- added joint link6NPP_link7NPP: type revolute, parent link6NPP, child link7NPP, origin xyz=-0.3412699882789874 0 0.24954597860926986 rpy=0 0 0, axis 1 0 0, limit lower=-3.14159 upper=3.14159 effort=0.0 velocity=0.0
- added joint rootLink_link1NNP: type revolute, parent rootLink, child link1NNP, origin xyz=0 -0.2 0.5 rpy=0 0 0, axis 0 1 0, limit lower=-3.14159 upper=3.14159 effort=0.0 velocity=0.0
- added joint rootLink_link1NPP: type revolute, parent rootLink, child link1NPP, origin xyz=0 0.2 0.5 rpy=0 0 0, axis 0 1 0, limit lower=-3.14159 upper=3.14159 effort=0.0 velocity=0.0

Commit message: a7: added pictures and edited readme

File: body.urdf (robot description, URDF)
Before this commit: robot robot, 15 links, 14 joints
Links:
- removed link link4NNP
- removed link link4NPP
- removed link link5NNP
- removed link link5NPP
- removed link link6NNP
- removed link link6NPP
- removed link link7NNP
- removed link link7NPP
- link link2NNP: geometry collision box size=0.4620132804055245 0.42393298353921244 0.2814361325595609; visual box size=0.4620132804055245 0.42393298353921244 0.2814361325595609
- link link2NPP: geometry collision box size=0.4620132804055245 0.42393298353921244 0.2814361325595609; visual box size=0.4620132804055245 0.42393298353921244 0.2814361325595609
- link link3NNP: geometry collision box size=0.9746704550624676 0.5881426513866996 0.7766587783510606; visual box size=0.9746704550624676 0.5881426513866996 0.7766587783510606
- link link3NPP: geometry collision box size=0.9746704550624676 0.5881426513866996 0.7766587783510606; visual box size=0.9746704550624676 0.5881426513866996 0.7766587783510606
- link rootLink: geometry collision box size=1 1 1; visual box size=1 1 1
Joints:
- removed joint link3NNP_link4NNP
- removed joint link3NPP_link4NPP
- removed joint link4NNP_link5NNP
- removed joint link4NPP_link5NPP
- removed joint link5NNP_link6NNP
- removed joint link5NPP_link6NPP
- removed joint link6NNP_link7NNP
- removed joint link6NPP_link7NPP
- joint link1NNP_link2NNP: axis 0 0 1 -> 1 0 0; origin xyz=0.0 0 0.5 rpy=0 0 0 -> xyz=0 0.0 0.5 rpy=0 0 0
- joint link1NPP_link2NPP: axis 0 0 1 -> 1 0 0; origin xyz=0.0 0 0.5 rpy=0 0 0 -> xyz=0 0.0 0.5 rpy=0 0 0
- joint link2NNP_link3NNP: axis 0 0 1 -> 0 1 0; origin xyz=-0.3749239354147129 0 0.44161916027528836 rpy=0 0 0 -> xyz=-0.23100664020276224 -0.21196649176960622 0 rpy=0 0 0
- joint link2NPP_link3NPP: axis 0 0 1 -> 0 1 0; origin xyz=-0.3749239354147129 0 0.44161916027528836 rpy=0 0 0 -> xyz=-0.23100664020276224 0.21196649176960622 0 rpy=0 0 0
- joint rootLink_link1NNP: origin xyz=0 -0.2 0.5 rpy=0 0 0 -> xyz=0 -0.5 0.5 rpy=0 0 0
- joint rootLink_link1NPP: origin xyz=0 0.2 0.5 rpy=0 0 0 -> xyz=0 0.5 0.5 rpy=0 0 0

Commit message: a7: added robot example and edited readme

File: body.urdf (robot description, URDF)
Before this commit: robot robot, 7 links, 6 joints
Links:
- added link link4NNP, mass 1; collision box size=0.5264379267707182 0.21626957543836292 0.6060662071896765; visual box size=0.5264379267707182 0.21626957543836292 0.6060662071896765
- added link link4NPP, mass 1; collision box size=0.5264379267707182 0.21626957543836292 0.6060662071896765; visual box size=0.5264379267707182 0.21626957543836292 0.6060662071896765
- added link link5NNP, mass 1; collision box size=0.4311487081764114 0.5331062800402171 0.27956527469121567; visual box size=0.4311487081764114 0.5331062800402171 0.27956527469121567
- added link link5NPP, mass 1; collision box size=0.4311487081764114 0.5331062800402171 0.27956527469121567; visual box size=0.4311487081764114 0.5331062800402171 0.27956527469121567
- added link link6NNP, mass 1; collision box size=0.26224410750927896 0.24131335124645467 0.9914215472178438; visual box size=0.26224410750927896 0.24131335124645467 0.9914215472178438
- added link link6NPP, mass 1; collision box size=0.26224410750927896 0.24131335124645467 0.9914215472178438; visual box size=0.26224410750927896 0.24131335124645467 0.9914215472178438
- link link2NNP: geometry collision box size=0.7227146843219301 0.42263693260679713 0.3539932750408252; visual box size=0.7227146843219301 0.42263693260679713 0.3539932750408252
- link link2NPP: geometry collision box size=0.7227146843219301 0.42263693260679713 0.3539932750408252; visual box size=0.7227146843219301 0.42263693260679713 0.3539932750408252
- link link3NNP: geometry collision box size=0.3587069385545301 0.5112295305766441 0.8030141248705229; visual box size=0.3587069385545301 0.5112295305766441 0.8030141248705229
- link link3NPP: geometry collision box size=0.3587069385545301 0.5112295305766441 0.8030141248705229; visual box size=0.3587069385545301 0.5112295305766441 0.8030141248705229
Joints:
- added joint link3NNP_link4NNP: type revolute, parent link3NNP, child link4NNP, origin xyz=0 -0.25561476528832205 0.40150706243526146 rpy=0 0 0, axis 0 0 1, limit lower=-3.14159 upper=3.14159 effort=0.0 velocity=0.0
- added joint link3NPP_link4NPP: type revolute, parent link3NPP, child link4NPP, origin xyz=0 0.25561476528832205 0.40150706243526146 rpy=0 0 0, axis 0 0 1, limit lower=-3.14159 upper=3.14159 effort=0.0 velocity=0.0
- added joint link4NNP_link5NNP: type revolute, parent link4NNP, child link5NNP, origin xyz=-0.2632189633853591 0 0.30303310359483826 rpy=0 0 0, axis 1 0 0, limit lower=-3.14159 upper=3.14159 effort=0.0 velocity=0.0
- added joint link4NPP_link5NPP: type revolute, parent link4NPP, child link5NPP, origin xyz=-0.2632189633853591 0 0.30303310359483826 rpy=0 0 0, axis 1 0 0, limit lower=-3.14159 upper=3.14159 effort=0.0 velocity=0.0
- added joint link5NNP_link6NNP: type revolute, parent link5NNP, child link6NNP, origin xyz=-0.2155743540882057 -0.26655314002010855 0 rpy=0 0 0, axis 0 0 1, limit lower=-3.14159 upper=3.14159 effort=0.0 velocity=0.0
- added joint link5NPP_link6NPP: type revolute, parent link5NPP, child link6NPP, origin xyz=-0.2155743540882057 0.26655314002010855 0 rpy=0 0 0, axis 0 0 1, limit lower=-3.14159 upper=3.14159 effort=0.0 velocity=0.0
- joint link1NNP_link2NNP: origin xyz=0 0.0 0.5 rpy=0 0 0 -> xyz=0.0 0 0.5 rpy=0 0 0
- joint link1NPP_link2NPP: origin xyz=0 0.0 0.5 rpy=0 0 0 -> xyz=0.0 0 0.5 rpy=0 0 0
- joint link2NNP_link3NNP: origin xyz=-0.23100664020276224 -0.21196649176960622 0 rpy=0 0 0 -> xyz=-0.36135734216096504 -0.21131846630339857 0 rpy=0 0 0
- joint link2NPP_link3NPP: origin xyz=-0.23100664020276224 0.21196649176960622 0 rpy=0 0 0 -> xyz=-0.36135734216096504 0.21131846630339857 0 rpy=0 0 0
