Commit message: a7:

File: body.urdf (robot description, URDF)
Before this commit: robot robot, 13 links, 12 joints
Links:
- removed link link6NNP
- removed link link6NPP
- link link2NNP: geometry collision box size=0.8101265621398726 0.24644277798984673 0.7784325727808661; visual box size=0.8101265621398726 0.24644277798984673 0.7784325727808661
- link link2NPP: geometry collision box size=0.8101265621398726 0.24644277798984673 0.7784325727808661; visual box size=0.8101265621398726 0.24644277798984673 0.7784325727808661
- link link3NNP: geometry collision box size=0.9184821836643737 0.39918190564402145 0.8345910579732303; visual box size=0.9184821836643737 0.39918190564402145 0.8345910579732303
- link link3NPP: geometry collision box size=0.9184821836643737 0.39918190564402145 0.8345910579732303; visual box size=0.9184821836643737 0.39918190564402145 0.8345910579732303
- link link4NNP: geometry collision box size=0.3039231997022676 0.31605218893191744 0.3280574522338664; visual box size=0.3039231997022676 0.31605218893191744 0.3280574522338664
- link link4NPP: geometry collision box size=0.3039231997022676 0.31605218893191744 0.3280574522338664; visual box size=0.3039231997022676 0.31605218893191744 0.3280574522338664
- link link5NNP: geometry collision box size=0.7437661336207813 0.3388128057670559 0.22177063077538542; visual box size=0.7437661336207813 0.3388128057670559 0.22177063077538542
- link link5NPP: geometry collision box size=0.7437661336207813 0.3388128057670559 0.22177063077538542; visual box size=0.7437661336207813 0.3388128057670559 0.22177063077538542
Joints:
- removed joint link5NNP_link6NNP
- removed joint link5NPP_link6NPP
- joint link2NNP_link3NNP: origin xyz=-0.36135734216096504 -0.21131846630339857 0 rpy=0 0 0 -> xyz=-0.4050632810699363 -0.12322138899492337 0 rpy=0 0 0
- joint link2NPP_link3NPP: origin xyz=-0.36135734216096504 0.21131846630339857 0 rpy=0 0 0 -> xyz=-0.4050632810699363 0.12322138899492337 0 rpy=0 0 0
- joint link3NNP_link4NNP: axis 0 0 1 -> 1 0 0; origin xyz=0 -0.25561476528832205 0.40150706243526146 rpy=0 0 0 -> xyz=0 -0.19959095282201073 0.41729552898661515 rpy=0 0 0
- joint link3NPP_link4NPP: axis 0 0 1 -> 1 0 0; origin xyz=0 0.25561476528832205 0.40150706243526146 rpy=0 0 0 -> xyz=0 0.19959095282201073 0.41729552898661515 rpy=0 0 0
- joint link4NNP_link5NNP: origin xyz=-0.2632189633853591 0 0.30303310359483826 rpy=0 0 0 -> xyz=0 -0.15802609446595872 0.1640287261169332 rpy=0 0 0
- joint link4NPP_link5NPP: origin xyz=-0.2632189633853591 0 0.30303310359483826 rpy=0 0 0 -> xyz=0 0.15802609446595872 0.1640287261169332 rpy=0 0 0

Commit message: a8: fixed up solution.py....

File: body.urdf (robot description, URDF)
Before this commit: robot robot, 11 links, 10 joints
Links:
- added link link6NNP, mass 1; collision box size=0.9898073608264104 0.4130254536354109 0.7641378033770159; visual box size=0.9898073608264104 0.4130254536354109 0.7641378033770159
- added link link6NPP, mass 1; collision box size=0.9898073608264104 0.4130254536354109 0.7641378033770159; visual box size=0.9898073608264104 0.4130254536354109 0.7641378033770159
- added link link7NNP, mass 1; collision box size=0.4481180554554661 0.4919326993040514 0.9190706303743947; visual box size=0.4481180554554661 0.4919326993040514 0.9190706303743947
- added link link7NPP, mass 1; collision box size=0.4481180554554661 0.4919326993040514 0.9190706303743947; visual box size=0.4481180554554661 0.4919326993040514 0.9190706303743947
- link link2NNP: geometry collision box size=0.8063635223522421 0.368228632332338 0.4071334002343707; visual box size=0.8063635223522421 0.368228632332338 0.4071334002343707
- link link2NPP: geometry collision box size=0.8063635223522421 0.368228632332338 0.4071334002343707; visual box size=0.8063635223522421 0.368228632332338 0.4071334002343707
- link link3NNP: geometry collision box size=0.5239473099603315 0.513519435613909 0.442650180863142; visual box size=0.5239473099603315 0.513519435613909 0.442650180863142
- link link3NPP: geometry collision box size=0.5239473099603315 0.513519435613909 0.442650180863142; visual box size=0.5239473099603315 0.513519435613909 0.442650180863142
- link link4NNP: geometry collision box size=0.48643949975599066 0.556664263928273 0.37475418153218537; visual box size=0.48643949975599066 0.556664263928273 0.37475418153218537
- link link4NPP: geometry collision box size=0.48643949975599066 0.556664263928273 0.37475418153218537; visual box size=0.48643949975599066 0.556664263928273 0.37475418153218537
- link link5NNP: geometry collision box size=0.4254702755197631 0.5023216816628895 0.6946951973402653; visual box size=0.4254702755197631 0.5023216816628895 0.6946951973402653
- link link5NPP: geometry collision box size=0.4254702755197631 0.5023216816628895 0.6946951973402653; visual box size=0.4254702755197631 0.5023216816628895 0.6946951973402653
Joints:
- added joint link5NNP_link6NNP: type revolute, parent link5NNP, child link6NNP, origin xyz=-0.21273513775988154 0 0.34734759867013265 rpy=0 0 0, axis 0 1 0, limit lower=-3.14159 upper=3.14159 effort=0.0 velocity=0.0
- added joint link5NPP_link6NPP: type revolute, parent link5NPP, child link6NPP, origin xyz=-0.21273513775988154 0 0.34734759867013265 rpy=0 0 0, axis 0 1 0, limit lower=-3.14159 upper=3.14159 effort=0.0 velocity=0.0
- added joint link6NNP_link7NNP: type revolute, parent link6NNP, child link7NNP, origin xyz=-0.4949036804132052 -0.20651272681770544 0 rpy=0 0 0, axis 1 0 0, limit lower=-3.14159 upper=3.14159 effort=0.0 velocity=0.0
- added joint link6NPP_link7NPP: type revolute, parent link6NPP, child link7NPP, origin xyz=-0.4949036804132052 0.20651272681770544 0 rpy=0 0 0, axis 1 0 0, limit lower=-3.14159 upper=3.14159 effort=0.0 velocity=0.0
- joint link1NNP_link2NNP: axis 1 0 0 -> 0 0 1; origin xyz=0.0 0 0.5 rpy=0 0 0 -> xyz=0 0.0 0.5 rpy=0 0 0
- joint link1NPP_link2NPP: axis 1 0 0 -> 0 0 1; origin xyz=0.0 0 0.5 rpy=0 0 0 -> xyz=0 0.0 0.5 rpy=0 0 0
- joint link2NNP_link3NNP: origin xyz=-0.4050632810699363 -0.12322138899492337 0 rpy=0 0 0 -> xyz=0 -0.184114316166169 0.20356670011718536 rpy=0 0 0
- joint link2NPP_link3NPP: origin xyz=-0.4050632810699363 0.12322138899492337 0 rpy=0 0 0 -> xyz=0 0.184114316166169 0.20356670011718536 rpy=0 0 0
- joint link3NNP_link4NNP: axis 1 0 0 -> 0 1 0; origin xyz=0 -0.19959095282201073 0.41729552898661515 rpy=0 0 0 -> xyz=-0.2619736549801657 0 0.221325090431571 rpy=0 0 0
- joint link3NPP_link4NPP: axis 1 0 0 -> 0 1 0; origin xyz=0 0.19959095282201073 0.41729552898661515 rpy=0 0 0 -> xyz=-0.2619736549801657 0 0.221325090431571 rpy=0 0 0
- joint link4NNP_link5NNP: axis 1 0 0 -> 0 0 1; origin xyz=0 -0.15802609446595872 0.1640287261169332 rpy=0 0 0 -> xyz=-0.24321974987799533 0 0.18737709076609269 rpy=0 0 0
- joint link4NPP_link5NPP: axis 1 0 0 -> 0 0 1; origin xyz=0 0.15802609446595872 0.1640287261169332 rpy=0 0 0 -> xyz=-0.24321974987799533 0 0.18737709076609269 rpy=0 0 0
