Commit message: a8: lookin pretty good. done with graphs. need to mutate function and deal with file mgmt and show best

File: body12.urdf (robot description, URDF)
Before this commit: robot robot, 11 links, 10 joints
Links:
- added link link6NNP, mass 1; collision box size=0.9898073608264104 0.4130254536354109 0.7641378033770159; visual box size=0.9898073608264104 0.4130254536354109 0.7641378033770159
- added link link6NPP, mass 1; collision box size=0.9898073608264104 0.4130254536354109 0.7641378033770159; visual box size=0.9898073608264104 0.4130254536354109 0.7641378033770159
- added link link7NNP, mass 1; collision box size=0.4481180554554661 0.4919326993040514 0.9190706303743947; visual box size=0.4481180554554661 0.4919326993040514 0.9190706303743947
- added link link7NPP, mass 1; collision box size=0.4481180554554661 0.4919326993040514 0.9190706303743947; visual box size=0.4481180554554661 0.4919326993040514 0.9190706303743947
- link link2NNP: geometry collision box size=0.8063635223522421 0.368228632332338 0.4071334002343707; visual box size=0.8063635223522421 0.368228632332338 0.4071334002343707
- link link2NPP: geometry collision box size=0.8063635223522421 0.368228632332338 0.4071334002343707; visual box size=0.8063635223522421 0.368228632332338 0.4071334002343707
- link link3NNP: geometry collision box size=0.5239473099603315 0.513519435613909 0.442650180863142; visual box size=0.5239473099603315 0.513519435613909 0.442650180863142
- link link3NPP: geometry collision box size=0.5239473099603315 0.513519435613909 0.442650180863142; visual box size=0.5239473099603315 0.513519435613909 0.442650180863142
- link link4NNP: geometry collision box size=0.48643949975599066 0.556664263928273 0.37475418153218537; visual box size=0.48643949975599066 0.556664263928273 0.37475418153218537
- link link4NPP: geometry collision box size=0.48643949975599066 0.556664263928273 0.37475418153218537; visual box size=0.48643949975599066 0.556664263928273 0.37475418153218537
- link link5NNP: geometry collision box size=0.4254702755197631 0.5023216816628895 0.6946951973402653; visual box size=0.4254702755197631 0.5023216816628895 0.6946951973402653
- link link5NPP: geometry collision box size=0.4254702755197631 0.5023216816628895 0.6946951973402653; visual box size=0.4254702755197631 0.5023216816628895 0.6946951973402653
Joints:
- added joint link5NNP_link6NNP: type revolute, parent link5NNP, child link6NNP, origin xyz=-0.21273513775988154 0 0.34734759867013265 rpy=0 0 0, axis 0 1 0, limit lower=-3.14159 upper=3.14159 effort=0.0 velocity=0.0
- added joint link5NPP_link6NPP: type revolute, parent link5NPP, child link6NPP, origin xyz=-0.21273513775988154 0 0.34734759867013265 rpy=0 0 0, axis 0 1 0, limit lower=-3.14159 upper=3.14159 effort=0.0 velocity=0.0
- added joint link6NNP_link7NNP: type revolute, parent link6NNP, child link7NNP, origin xyz=-0.4949036804132052 -0.20651272681770544 0 rpy=0 0 0, axis 1 0 0, limit lower=-3.14159 upper=3.14159 effort=0.0 velocity=0.0
- added joint link6NPP_link7NPP: type revolute, parent link6NPP, child link7NPP, origin xyz=-0.4949036804132052 0.20651272681770544 0 rpy=0 0 0, axis 1 0 0, limit lower=-3.14159 upper=3.14159 effort=0.0 velocity=0.0
- joint link1NNP_link2NNP: axis 1 0 0 -> 0 0 1; origin xyz=0.0 0 0.5 rpy=0 0 0 -> xyz=0 0.0 0.5 rpy=0 0 0
- joint link1NPP_link2NPP: axis 1 0 0 -> 0 0 1; origin xyz=0.0 0 0.5 rpy=0 0 0 -> xyz=0 0.0 0.5 rpy=0 0 0
- joint link2NNP_link3NNP: origin xyz=-0.22131943435420404 0 0.29155135796955906 rpy=0 0 0 -> xyz=0 -0.184114316166169 0.20356670011718536 rpy=0 0 0
- joint link2NPP_link3NPP: origin xyz=-0.22131943435420404 0 0.29155135796955906 rpy=0 0 0 -> xyz=0 0.184114316166169 0.20356670011718536 rpy=0 0 0
- joint link3NNP_link4NNP: origin xyz=-0.12660603827183597 0 0.46718201723508757 rpy=0 0 0 -> xyz=-0.2619736549801657 0 0.221325090431571 rpy=0 0 0
- joint link3NPP_link4NPP: origin xyz=-0.12660603827183597 0 0.46718201723508757 rpy=0 0 0 -> xyz=-0.2619736549801657 0 0.221325090431571 rpy=0 0 0
- joint link4NNP_link5NNP: origin xyz=-0.18877127027612706 -0.20733600163496269 0 rpy=0 0 0 -> xyz=-0.24321974987799533 0 0.18737709076609269 rpy=0 0 0
- joint link4NPP_link5NPP: origin xyz=-0.18877127027612706 0.20733600163496269 0 rpy=0 0 0 -> xyz=-0.24321974987799533 0 0.18737709076609269 rpy=0 0 0

File: body13.urdf (robot description, URDF)
Before this commit: robot robot, 11 links, 10 joints
Links:
- added link link6NNP, mass 1; collision box size=0.8515734906330688 0.41611344278812956 0.9710708367790408; visual box size=0.8515734906330688 0.41611344278812956 0.9710708367790408
- added link link6NPP, mass 1; collision box size=0.8515734906330688 0.41611344278812956 0.9710708367790408; visual box size=0.8515734906330688 0.41611344278812956 0.9710708367790408
- link link2NNP: geometry collision box size=0.7629140369324161 0.22519370970447983 0.9336151752919599; visual box size=0.7629140369324161 0.22519370970447983 0.9336151752919599
- link link2NPP: geometry collision box size=0.7629140369324161 0.22519370970447983 0.9336151752919599; visual box size=0.7629140369324161 0.22519370970447983 0.9336151752919599
- link link3NNP: geometry collision box size=0.3908927428921762 0.5870161001160573 0.8425435754238961; visual box size=0.3908927428921762 0.5870161001160573 0.8425435754238961
- link link3NPP: geometry collision box size=0.3908927428921762 0.5870161001160573 0.8425435754238961; visual box size=0.3908927428921762 0.5870161001160573 0.8425435754238961
- link link4NNP: geometry collision box size=0.2729727630641807 0.5972886214257913 0.9000698298689165; visual box size=0.2729727630641807 0.5972886214257913 0.9000698298689165
- link link4NPP: geometry collision box size=0.2729727630641807 0.5972886214257913 0.9000698298689165; visual box size=0.2729727630641807 0.5972886214257913 0.9000698298689165
- link link5NNP: geometry collision box size=0.28724627674488296 0.42050689843622047 0.7652491278935118; visual box size=0.28724627674488296 0.42050689843622047 0.7652491278935118
- link link5NPP: geometry collision box size=0.28724627674488296 0.42050689843622047 0.7652491278935118; visual box size=0.28724627674488296 0.42050689843622047 0.7652491278935118
Joints:
- added joint link5NNP_link6NNP: type revolute, parent link5NNP, child link6NNP, origin xyz=0 -0.21025344921811023 0.3826245639467559 rpy=0 0 0, axis 1 0 0, limit lower=-3.14159 upper=3.14159 effort=0.0 velocity=0.0
- added joint link5NPP_link6NPP: type revolute, parent link5NPP, child link6NPP, origin xyz=0 0.21025344921811023 0.3826245639467559 rpy=0 0 0, axis 1 0 0, limit lower=-3.14159 upper=3.14159 effort=0.0 velocity=0.0
- joint link1NNP_link2NNP: axis 0 0 1 -> 0 1 0; origin xyz=0 0.0 0.5 rpy=0 0 0 -> xyz=0.0 0 0.5 rpy=0 0 0
- joint link1NPP_link2NPP: axis 0 0 1 -> 0 1 0; origin xyz=0 0.0 0.5 rpy=0 0 0 -> xyz=0.0 0 0.5 rpy=0 0 0
- joint link2NNP_link3NNP: axis 0 1 0 -> 1 0 0; origin xyz=0 -0.15599951906404824 0.47783111612376084 rpy=0 0 0 -> xyz=-0.38145701846620805 -0.11259685485223991 0 rpy=0 0 0
- joint link2NPP_link3NPP: axis 0 1 0 -> 1 0 0; origin xyz=0 0.15599951906404824 0.47783111612376084 rpy=0 0 0 -> xyz=-0.38145701846620805 0.11259685485223991 0 rpy=0 0 0
- joint link3NNP_link4NNP: origin xyz=-0.10288453372976268 0 0.38196277583336 rpy=0 0 0 -> xyz=0 -0.29350805005802866 0.42127178771194806 rpy=0 0 0
- joint link3NPP_link4NPP: origin xyz=-0.10288453372976268 0 0.38196277583336 rpy=0 0 0 -> xyz=0 0.29350805005802866 0.42127178771194806 rpy=0 0 0
- joint link4NNP_link5NNP: axis 0 0 1 -> 1 0 0; origin xyz=-0.4392176352894539 0 0.2655784172526928 rpy=0 0 0 -> xyz=0 -0.29864431071289566 0.45003491493445824 rpy=0 0 0
- joint link4NPP_link5NPP: axis 0 0 1 -> 1 0 0; origin xyz=-0.4392176352894539 0 0.2655784172526928 rpy=0 0 0 -> xyz=0 0.29864431071289566 0.45003491493445824 rpy=0 0 0

File: body15.urdf (robot description, URDF)
Before this commit: robot robot, 11 links, 10 joints
Links:
- added link link6NNP, mass 1; collision box size=0.9898073608264104 0.4130254536354109 0.7641378033770159; visual box size=0.9898073608264104 0.4130254536354109 0.7641378033770159
- added link link6NPP, mass 1; collision box size=0.9898073608264104 0.4130254536354109 0.7641378033770159; visual box size=0.9898073608264104 0.4130254536354109 0.7641378033770159
- added link link7NNP, mass 1; collision box size=0.4481180554554661 0.4919326993040514 0.9190706303743947; visual box size=0.4481180554554661 0.4919326993040514 0.9190706303743947
- added link link7NPP, mass 1; collision box size=0.4481180554554661 0.4919326993040514 0.9190706303743947; visual box size=0.4481180554554661 0.4919326993040514 0.9190706303743947
- link link2NNP: geometry collision box size=0.8063635223522421 0.368228632332338 0.4071334002343707; visual box size=0.8063635223522421 0.368228632332338 0.4071334002343707
- link link2NPP: geometry collision box size=0.8063635223522421 0.368228632332338 0.4071334002343707; visual box size=0.8063635223522421 0.368228632332338 0.4071334002343707
- link link3NNP: geometry collision box size=0.5239473099603315 0.513519435613909 0.442650180863142; visual box size=0.5239473099603315 0.513519435613909 0.442650180863142
- link link3NPP: geometry collision box size=0.5239473099603315 0.513519435613909 0.442650180863142; visual box size=0.5239473099603315 0.513519435613909 0.442650180863142
- link link4NNP: geometry collision box size=0.48643949975599066 0.556664263928273 0.37475418153218537; visual box size=0.48643949975599066 0.556664263928273 0.37475418153218537
- link link4NPP: geometry collision box size=0.48643949975599066 0.556664263928273 0.37475418153218537; visual box size=0.48643949975599066 0.556664263928273 0.37475418153218537
- link link5NNP: geometry collision box size=0.4254702755197631 0.5023216816628895 0.6946951973402653; visual box size=0.4254702755197631 0.5023216816628895 0.6946951973402653
- link link5NPP: geometry collision box size=0.4254702755197631 0.5023216816628895 0.6946951973402653; visual box size=0.4254702755197631 0.5023216816628895 0.6946951973402653
Joints:
- added joint link5NNP_link6NNP: type revolute, parent link5NNP, child link6NNP, origin xyz=-0.21273513775988154 0 0.34734759867013265 rpy=0 0 0, axis 0 1 0, limit lower=-3.14159 upper=3.14159 effort=0.0 velocity=0.0
- added joint link5NPP_link6NPP: type revolute, parent link5NPP, child link6NPP, origin xyz=-0.21273513775988154 0 0.34734759867013265 rpy=0 0 0, axis 0 1 0, limit lower=-3.14159 upper=3.14159 effort=0.0 velocity=0.0
- added joint link6NNP_link7NNP: type revolute, parent link6NNP, child link7NNP, origin xyz=-0.4949036804132052 -0.20651272681770544 0 rpy=0 0 0, axis 1 0 0, limit lower=-3.14159 upper=3.14159 effort=0.0 velocity=0.0
- added joint link6NPP_link7NPP: type revolute, parent link6NPP, child link7NPP, origin xyz=-0.4949036804132052 0.20651272681770544 0 rpy=0 0 0, axis 1 0 0, limit lower=-3.14159 upper=3.14159 effort=0.0 velocity=0.0
- joint link1NNP_link2NNP: axis 1 0 0 -> 0 0 1; origin xyz=0.0 0 0.5 rpy=0 0 0 -> xyz=0 0.0 0.5 rpy=0 0 0
- joint link1NPP_link2NPP: axis 1 0 0 -> 0 0 1; origin xyz=0.0 0 0.5 rpy=0 0 0 -> xyz=0 0.0 0.5 rpy=0 0 0
- joint link2NNP_link3NNP: origin xyz=-0.22131943435420404 0 0.29155135796955906 rpy=0 0 0 -> xyz=0 -0.184114316166169 0.20356670011718536 rpy=0 0 0
- joint link2NPP_link3NPP: origin xyz=-0.22131943435420404 0 0.29155135796955906 rpy=0 0 0 -> xyz=0 0.184114316166169 0.20356670011718536 rpy=0 0 0
- joint link3NNP_link4NNP: origin xyz=-0.12660603827183597 0 0.46718201723508757 rpy=0 0 0 -> xyz=-0.2619736549801657 0 0.221325090431571 rpy=0 0 0
- joint link3NPP_link4NPP: origin xyz=-0.12660603827183597 0 0.46718201723508757 rpy=0 0 0 -> xyz=-0.2619736549801657 0 0.221325090431571 rpy=0 0 0
- joint link4NNP_link5NNP: origin xyz=-0.18877127027612706 -0.20733600163496269 0 rpy=0 0 0 -> xyz=-0.24321974987799533 0 0.18737709076609269 rpy=0 0 0
- joint link4NPP_link5NPP: origin xyz=-0.18877127027612706 0.20733600163496269 0 rpy=0 0 0 -> xyz=-0.24321974987799533 0 0.18737709076609269 rpy=0 0 0

File: body17.urdf (robot description, URDF)
Before this commit: robot robot, 13 links, 12 joints
Links:
- removed link link5NNP
- removed link link5NPP
- removed link link6NNP
- removed link link6NPP
- link link2NNP: geometry collision box size=0.873968178512146 0.5592692485431516 0.9384659518561416; visual box size=0.873968178512146 0.5592692485431516 0.9384659518561416
- link link2NPP: geometry collision box size=0.873968178512146 0.5592692485431516 0.9384659518561416; visual box size=0.873968178512146 0.5592692485431516 0.9384659518561416
- link link3NNP: geometry collision box size=0.8702921849804126 0.40982957564483313 0.6174320805765909; visual box size=0.8702921849804126 0.40982957564483313 0.6174320805765909
- link link3NPP: geometry collision box size=0.8702921849804126 0.40982957564483313 0.6174320805765909; visual box size=0.8702921849804126 0.40982957564483313 0.6174320805765909
- link link4NNP: geometry collision box size=0.8795887721490938 0.55801558697067 0.6718409468249279; visual box size=0.8795887721490938 0.55801558697067 0.6718409468249279
- link link4NPP: geometry collision box size=0.8795887721490938 0.55801558697067 0.6718409468249279; visual box size=0.8795887721490938 0.55801558697067 0.6718409468249279
Joints:
- removed joint link4NNP_link5NNP
- removed joint link4NPP_link5NPP
- removed joint link5NNP_link6NNP
- removed joint link5NPP_link6NPP
- joint link1NNP_link2NNP: axis 0 1 0 -> 1 0 0
- joint link1NPP_link2NPP: axis 0 1 0 -> 1 0 0
- joint link2NNP_link3NNP: axis 1 0 0 -> 0 1 0; origin xyz=-0.1734814594859801 -0.18718486688575547 0 rpy=0 0 0 -> xyz=-0.436984089256073 -0.2796346242715758 0 rpy=0 0 0
- joint link2NPP_link3NPP: axis 1 0 0 -> 0 1 0; origin xyz=-0.1734814594859801 0.18718486688575547 0 rpy=0 0 0 -> xyz=-0.436984089256073 0.2796346242715758 0 rpy=0 0 0
- joint link3NNP_link4NNP: origin xyz=-0.4617260406122631 0 0.12464409681607035 rpy=0 0 0 -> xyz=-0.4351460924902063 -0.20491478782241657 0 rpy=0 0 0
- joint link3NPP_link4NPP: origin xyz=-0.4617260406122631 0 0.12464409681607035 rpy=0 0 0 -> xyz=-0.4351460924902063 0.20491478782241657 0 rpy=0 0 0

File: body2.urdf (robot description, URDF)
Before this commit: robot robot, 13 links, 12 joints
Links:
- removed link link5NNP
- removed link link5NPP
- removed link link6NNP
- removed link link6NPP
- link link2NNP: geometry collision box size=0.873968178512146 0.5592692485431516 0.9384659518561416; visual box size=0.873968178512146 0.5592692485431516 0.9384659518561416
- link link2NPP: geometry collision box size=0.873968178512146 0.5592692485431516 0.9384659518561416; visual box size=0.873968178512146 0.5592692485431516 0.9384659518561416
- link link3NNP: geometry collision box size=0.8702921849804126 0.40982957564483313 0.6174320805765909; visual box size=0.8702921849804126 0.40982957564483313 0.6174320805765909
- link link3NPP: geometry collision box size=0.8702921849804126 0.40982957564483313 0.6174320805765909; visual box size=0.8702921849804126 0.40982957564483313 0.6174320805765909
- link link4NNP: geometry collision box size=0.8795887721490938 0.55801558697067 0.6718409468249279; visual box size=0.8795887721490938 0.55801558697067 0.6718409468249279
- link link4NPP: geometry collision box size=0.8795887721490938 0.55801558697067 0.6718409468249279; visual box size=0.8795887721490938 0.55801558697067 0.6718409468249279
Joints:
- removed joint link4NNP_link5NNP
- removed joint link4NPP_link5NPP
- removed joint link5NNP_link6NNP
- removed joint link5NPP_link6NPP
- joint link1NNP_link2NNP: axis 0 1 0 -> 1 0 0
- joint link1NPP_link2NPP: axis 0 1 0 -> 1 0 0
- joint link2NNP_link3NNP: axis 1 0 0 -> 0 1 0; origin xyz=-0.1734814594859801 -0.18718486688575547 0 rpy=0 0 0 -> xyz=-0.436984089256073 -0.2796346242715758 0 rpy=0 0 0
- joint link2NPP_link3NPP: axis 1 0 0 -> 0 1 0; origin xyz=-0.1734814594859801 0.18718486688575547 0 rpy=0 0 0 -> xyz=-0.436984089256073 0.2796346242715758 0 rpy=0 0 0
- joint link3NNP_link4NNP: origin xyz=-0.4617260406122631 0 0.12464409681607035 rpy=0 0 0 -> xyz=-0.4351460924902063 -0.20491478782241657 0 rpy=0 0 0
- joint link3NPP_link4NPP: origin xyz=-0.4617260406122631 0 0.12464409681607035 rpy=0 0 0 -> xyz=-0.4351460924902063 0.20491478782241657 0 rpy=0 0 0

File: body3.urdf (robot description, URDF)
Before this commit: robot robot, 11 links, 10 joints
Links:
- added link link6NNP, mass 1; collision box size=0.9898073608264104 0.4130254536354109 0.7641378033770159; visual box size=0.9898073608264104 0.4130254536354109 0.7641378033770159
- added link link6NPP, mass 1; collision box size=0.9898073608264104 0.4130254536354109 0.7641378033770159; visual box size=0.9898073608264104 0.4130254536354109 0.7641378033770159
- added link link7NNP, mass 1; collision box size=0.4481180554554661 0.4919326993040514 0.9190706303743947; visual box size=0.4481180554554661 0.4919326993040514 0.9190706303743947
- added link link7NPP, mass 1; collision box size=0.4481180554554661 0.4919326993040514 0.9190706303743947; visual box size=0.4481180554554661 0.4919326993040514 0.9190706303743947
- link link2NNP: geometry collision box size=0.8063635223522421 0.368228632332338 0.4071334002343707; visual box size=0.8063635223522421 0.368228632332338 0.4071334002343707
- link link2NPP: geometry collision box size=0.8063635223522421 0.368228632332338 0.4071334002343707; visual box size=0.8063635223522421 0.368228632332338 0.4071334002343707
- link link3NNP: geometry collision box size=0.5239473099603315 0.513519435613909 0.442650180863142; visual box size=0.5239473099603315 0.513519435613909 0.442650180863142
- link link3NPP: geometry collision box size=0.5239473099603315 0.513519435613909 0.442650180863142; visual box size=0.5239473099603315 0.513519435613909 0.442650180863142
- link link4NNP: geometry collision box size=0.48643949975599066 0.556664263928273 0.37475418153218537; visual box size=0.48643949975599066 0.556664263928273 0.37475418153218537
- link link4NPP: geometry collision box size=0.48643949975599066 0.556664263928273 0.37475418153218537; visual box size=0.48643949975599066 0.556664263928273 0.37475418153218537
- link link5NNP: geometry collision box size=0.4254702755197631 0.5023216816628895 0.6946951973402653; visual box size=0.4254702755197631 0.5023216816628895 0.6946951973402653
- link link5NPP: geometry collision box size=0.4254702755197631 0.5023216816628895 0.6946951973402653; visual box size=0.4254702755197631 0.5023216816628895 0.6946951973402653
Joints:
- added joint link5NNP_link6NNP: type revolute, parent link5NNP, child link6NNP, origin xyz=-0.21273513775988154 0 0.34734759867013265 rpy=0 0 0, axis 0 1 0, limit lower=-3.14159 upper=3.14159 effort=0.0 velocity=0.0
- added joint link5NPP_link6NPP: type revolute, parent link5NPP, child link6NPP, origin xyz=-0.21273513775988154 0 0.34734759867013265 rpy=0 0 0, axis 0 1 0, limit lower=-3.14159 upper=3.14159 effort=0.0 velocity=0.0
- added joint link6NNP_link7NNP: type revolute, parent link6NNP, child link7NNP, origin xyz=-0.4949036804132052 -0.20651272681770544 0 rpy=0 0 0, axis 1 0 0, limit lower=-3.14159 upper=3.14159 effort=0.0 velocity=0.0
- added joint link6NPP_link7NPP: type revolute, parent link6NPP, child link7NPP, origin xyz=-0.4949036804132052 0.20651272681770544 0 rpy=0 0 0, axis 1 0 0, limit lower=-3.14159 upper=3.14159 effort=0.0 velocity=0.0
- joint link1NNP_link2NNP: axis 1 0 0 -> 0 0 1; origin xyz=0.0 0 0.5 rpy=0 0 0 -> xyz=0 0.0 0.5 rpy=0 0 0
- joint link1NPP_link2NPP: axis 1 0 0 -> 0 0 1; origin xyz=0.0 0 0.5 rpy=0 0 0 -> xyz=0 0.0 0.5 rpy=0 0 0
- joint link2NNP_link3NNP: origin xyz=-0.22131943435420404 0 0.29155135796955906 rpy=0 0 0 -> xyz=0 -0.184114316166169 0.20356670011718536 rpy=0 0 0
- joint link2NPP_link3NPP: origin xyz=-0.22131943435420404 0 0.29155135796955906 rpy=0 0 0 -> xyz=0 0.184114316166169 0.20356670011718536 rpy=0 0 0
- joint link3NNP_link4NNP: origin xyz=-0.12660603827183597 0 0.46718201723508757 rpy=0 0 0 -> xyz=-0.2619736549801657 0 0.221325090431571 rpy=0 0 0
- joint link3NPP_link4NPP: origin xyz=-0.12660603827183597 0 0.46718201723508757 rpy=0 0 0 -> xyz=-0.2619736549801657 0 0.221325090431571 rpy=0 0 0
- joint link4NNP_link5NNP: origin xyz=-0.18877127027612706 -0.20733600163496269 0 rpy=0 0 0 -> xyz=-0.24321974987799533 0 0.18737709076609269 rpy=0 0 0
- joint link4NPP_link5NPP: origin xyz=-0.18877127027612706 0.20733600163496269 0 rpy=0 0 0 -> xyz=-0.24321974987799533 0 0.18737709076609269 rpy=0 0 0
