Commit message: FP: figured out neuron counting issue; now show_best works!

File: body11.urdf (robot description, URDF)
Before this commit: robot robot, 9 links, 8 joints
Links:
- added link link5NNP, mass 1; collision box size=0.4254702755197631 0.5023216816628895 0.6946951973402653; visual box size=0.4254702755197631 0.5023216816628895 0.6946951973402653
- added link link5NPP, mass 1; collision box size=0.4254702755197631 0.5023216816628895 0.6946951973402653; visual box size=0.4254702755197631 0.5023216816628895 0.6946951973402653
Joints:
- added joint link4NNP_link5NNP: type revolute, parent link4NNP, child link5NNP, origin xyz=0 -0.2783321319641365 0.18737709076609269 rpy=0 0 0, axis 1 0 0, limit lower=-3.14159 upper=3.14159 effort=0.0 velocity=0.0
- added joint link4NPP_link5NPP: type revolute, parent link4NPP, child link5NPP, origin xyz=0 0.2783321319641365 0.18737709076609269 rpy=0 0 0, axis 1 0 0, limit lower=-3.14159 upper=3.14159 effort=0.0 velocity=0.0

File: body15.urdf (robot description, URDF)
Before this commit: robot robot, 9 links, 8 joints
Links:
- added link link5NNP, mass 1; collision box size=0.4254702755197631 0.5023216816628895 0.6946951973402653; visual box size=0.4254702755197631 0.5023216816628895 0.6946951973402653
- added link link5NPP, mass 1; collision box size=0.4254702755197631 0.5023216816628895 0.6946951973402653; visual box size=0.4254702755197631 0.5023216816628895 0.6946951973402653
Joints:
- added joint link4NNP_link5NNP: type revolute, parent link4NNP, child link5NNP, origin xyz=0 -0.2783321319641365 0.18737709076609269 rpy=0 0 0, axis 0 1 0, limit lower=-3.14159 upper=3.14159 effort=0.0 velocity=0.0
- added joint link4NPP_link5NPP: type revolute, parent link4NPP, child link5NPP, origin xyz=0 0.2783321319641365 0.18737709076609269 rpy=0 0 0, axis 0 1 0, limit lower=-3.14159 upper=3.14159 effort=0.0 velocity=0.0

File: body16.urdf (robot description, URDF)
Before this commit: robot robot, 9 links, 8 joints
Links:
- added link link5NNP, mass 1; collision box size=0.4254702755197631 0.5023216816628895 0.6946951973402653; visual box size=0.4254702755197631 0.5023216816628895 0.6946951973402653
- added link link5NPP, mass 1; collision box size=0.4254702755197631 0.5023216816628895 0.6946951973402653; visual box size=0.4254702755197631 0.5023216816628895 0.6946951973402653
Joints:
- added joint link4NNP_link5NNP: type revolute, parent link4NNP, child link5NNP, origin xyz=0 -0.2783321319641365 0.18737709076609269 rpy=0 0 0, axis 0 0 1, limit lower=-3.14159 upper=3.14159 effort=0.0 velocity=0.0
- added joint link4NPP_link5NPP: type revolute, parent link4NPP, child link5NPP, origin xyz=0 0.2783321319641365 0.18737709076609269 rpy=0 0 0, axis 0 0 1, limit lower=-3.14159 upper=3.14159 effort=0.0 velocity=0.0

File: body19.urdf (robot description, URDF)
Before this commit: robot robot, 9 links, 8 joints
Links:
- added link link5NNP, mass 1; collision box size=0.4254702755197631 0.5023216816628895 0.6946951973402653; visual box size=0.4254702755197631 0.5023216816628895 0.6946951973402653
- added link link5NPP, mass 1; collision box size=0.4254702755197631 0.5023216816628895 0.6946951973402653; visual box size=0.4254702755197631 0.5023216816628895 0.6946951973402653
Joints:
- added joint link4NNP_link5NNP: type revolute, parent link4NNP, child link5NNP, origin xyz=0 -0.2783321319641365 0.18737709076609269 rpy=0 0 0, axis 1 0 0, limit lower=-3.14159 upper=3.14159 effort=0.0 velocity=0.0
- added joint link4NPP_link5NPP: type revolute, parent link4NPP, child link5NPP, origin xyz=0 0.2783321319641365 0.18737709076609269 rpy=0 0 0, axis 1 0 0, limit lower=-3.14159 upper=3.14159 effort=0.0 velocity=0.0

File: body21.urdf (robot description, URDF)
Before this commit: robot robot, 9 links, 8 joints
Links:
- added link link5NNP, mass 1; collision box size=0.4254702755197631 0.5023216816628895 0.6946951973402653; visual box size=0.4254702755197631 0.5023216816628895 0.6946951973402653
- added link link5NPP, mass 1; collision box size=0.4254702755197631 0.5023216816628895 0.6946951973402653; visual box size=0.4254702755197631 0.5023216816628895 0.6946951973402653
Joints:
- added joint link4NNP_link5NNP: type revolute, parent link4NNP, child link5NNP, origin xyz=0 -0.2783321319641365 0.18737709076609269 rpy=0 0 0, axis 1 0 0, limit lower=-3.14159 upper=3.14159 effort=0.0 velocity=0.0
- added joint link4NPP_link5NPP: type revolute, parent link4NPP, child link5NPP, origin xyz=0 0.2783321319641365 0.18737709076609269 rpy=0 0 0, axis 1 0 0, limit lower=-3.14159 upper=3.14159 effort=0.0 velocity=0.0

File: body4.urdf (robot description, URDF)
Before this commit: robot robot, 9 links, 8 joints
Joints:
- joint link1NNP_link2NNP: axis 0 1 0 -> 0 0 1
- joint link1NPP_link2NPP: axis 0 1 0 -> 0 0 1

File: body5.urdf (robot description, URDF)
Before this commit: robot robot, 9 links, 8 joints
Joints:
- joint link2NNP_link3NNP: axis 0 0 1 -> 1 0 0
- joint link2NPP_link3NPP: axis 0 0 1 -> 1 0 0
