Commit message: FP: did two runs, added third hidden layer

File: body3.urdf (robot description, URDF)
Before this commit: robot robot, 9 links, 8 joints
Links:
- removed link link4NNP
- removed link link4NPP
- link link2NNP: geometry collision box size=0.6741127285017325 0.2521691184340571 0.932755849384785; visual box size=0.6741127285017325 0.2521691184340571 0.932755849384785
- link link2NPP: geometry collision box size=0.6741127285017325 0.2521691184340571 0.932755849384785; visual box size=0.6741127285017325 0.2521691184340571 0.932755849384785
- link link3NNP: geometry collision box size=0.7005762432864433 0.22621154369592525 0.21053439324389933; visual box size=0.7005762432864433 0.22621154369592525 0.21053439324389933
- link link3NPP: geometry collision box size=0.7005762432864433 0.22621154369592525 0.21053439324389933; visual box size=0.7005762432864433 0.22621154369592525 0.21053439324389933
Joints:
- removed joint link3NNP_link4NNP
- removed joint link3NPP_link4NPP
- joint link2NNP_link3NNP: origin xyz=-0.28885708618108535 0 0.2736687341815135 rpy=0 0 0 -> xyz=-0.33705636425086627 -0.12608455921702855 0 rpy=0 0 0
- joint link2NPP_link3NPP: origin xyz=-0.28885708618108535 0 0.2736687341815135 rpy=0 0 0 -> xyz=-0.33705636425086627 0.12608455921702855 0 rpy=0 0 0
