Commit message: a8: added new mutations

File: body0.urdf (robot description, URDF)
Before this commit: robot robot, 15 links, 14 joints
Links:
- removed link link4NNP
- removed link link4NPP
- removed link link5NNP
- removed link link5NPP
- removed link link6NNP
- removed link link6NPP
- removed link link7NNP
- removed link link7NPP
Joints:
- removed joint link3NNP_link4NNP
- removed joint link3NPP_link4NPP
- removed joint link4NNP_link5NNP
- removed joint link4NPP_link5NPP
- removed joint link5NNP_link6NNP
- removed joint link5NPP_link6NPP
- removed joint link6NNP_link7NNP
- removed joint link6NPP_link7NPP
- joint link1NNP_link2NNP: axis 0 0 1 -> 0 1 0
- joint link1NPP_link2NPP: axis 0 0 1 -> 0 1 0

File: body1.urdf (robot description, URDF)
Before this commit: robot robot, 13 links, 12 joints
Links:
- removed link link4NNP
- removed link link4NPP
- removed link link5NNP
- removed link link5NPP
- removed link link6NNP
- removed link link6NPP
- link link2NNP: geometry collision box size=0.8063635223522421 0.368228632332338 0.4071334002343707; visual box size=0.8063635223522421 0.368228632332338 0.4071334002343707
- link link2NPP: geometry collision box size=0.8063635223522421 0.368228632332338 0.4071334002343707; visual box size=0.8063635223522421 0.368228632332338 0.4071334002343707
- link link3NNP: geometry collision box size=0.5239473099603315 0.513519435613909 0.442650180863142; visual box size=0.5239473099603315 0.513519435613909 0.442650180863142
- link link3NPP: geometry collision box size=0.5239473099603315 0.513519435613909 0.442650180863142; visual box size=0.5239473099603315 0.513519435613909 0.442650180863142
Joints:
- removed joint link3NNP_link4NNP
- removed joint link3NPP_link4NPP
- removed joint link4NNP_link5NNP
- removed joint link4NPP_link5NPP
- removed joint link5NNP_link6NNP
- removed joint link5NPP_link6NPP
- joint link1NNP_link2NNP: origin xyz=0.0 0 0.5 rpy=0 0 0 -> xyz=0 0.0 0.5 rpy=0 0 0
- joint link1NPP_link2NPP: origin xyz=0.0 0 0.5 rpy=0 0 0 -> xyz=0 0.0 0.5 rpy=0 0 0
- joint link2NNP_link3NNP: axis 1 0 0 -> 0 1 0; origin xyz=-0.38145701846620805 -0.11259685485223991 0 rpy=0 0 0 -> xyz=0 -0.184114316166169 0.20356670011718536 rpy=0 0 0
- joint link2NPP_link3NPP: axis 1 0 0 -> 0 1 0; origin xyz=-0.38145701846620805 0.11259685485223991 0 rpy=0 0 0 -> xyz=0 0.184114316166169 0.20356670011718536 rpy=0 0 0

Commit message: a8: workin

File: body0.urdf (robot description, URDF)
Before this commit: robot robot, 7 links, 6 joints
Links:
- added link link4NNP, mass 1; collision box size=0.4019070140105776 0.40064106822721346 0.4539480724365998; visual box size=0.4019070140105776 0.40064106822721346 0.4539480724365998
- added link link4NPP, mass 1; collision box size=0.4019070140105776 0.40064106822721346 0.4539480724365998; visual box size=0.4019070140105776 0.40064106822721346 0.4539480724365998
- link link2NNP: geometry collision box size=0.8453526216949434 0.5841979097295507 0.4317003022115724; visual box size=0.8453526216949434 0.5841979097295507 0.4317003022115724
- link link2NPP: geometry collision box size=0.8453526216949434 0.5841979097295507 0.4317003022115724; visual box size=0.8453526216949434 0.5841979097295507 0.4317003022115724
- link link3NNP: geometry collision box size=0.2881296391337695 0.21077471151621074 0.5073368836354379; visual box size=0.2881296391337695 0.21077471151621074 0.5073368836354379
- link link3NPP: geometry collision box size=0.2881296391337695 0.21077471151621074 0.5073368836354379; visual box size=0.2881296391337695 0.21077471151621074 0.5073368836354379
Joints:
- added joint link3NNP_link4NNP: type revolute, parent link3NNP, child link4NNP, origin xyz=-0.14406481956688474 0 0.25366844181771897 rpy=0 0 0, axis 0 0 1, limit lower=-3.14159 upper=3.14159 effort=0.0 velocity=0.0
- added joint link3NPP_link4NPP: type revolute, parent link3NPP, child link4NPP, origin xyz=-0.14406481956688474 0 0.25366844181771897 rpy=0 0 0, axis 0 0 1, limit lower=-3.14159 upper=3.14159 effort=0.0 velocity=0.0
- joint link2NNP_link3NNP: axis 0 1 0 -> 1 0 0; origin xyz=0 -0.184114316166169 0.20356670011718536 rpy=0 0 0 -> xyz=-0.4226763108474717 -0.29209895486477533 0 rpy=0 0 0
- joint link2NPP_link3NPP: axis 0 1 0 -> 1 0 0; origin xyz=0 0.184114316166169 0.20356670011718536 rpy=0 0 0 -> xyz=-0.4226763108474717 0.29209895486477533 0 rpy=0 0 0
