Commit message: a8: working on readme

File: body5.urdf (robot description, URDF)
Before this commit: robot robot, 7 links, 6 joints
Links:
- added link link4NNP, mass 1; collision box size=0.8312712463921201 0.559507421379071 0.518589386631407; visual box size=0.8312712463921201 0.559507421379071 0.518589386631407
- added link link4NPP, mass 1; collision box size=0.8312712463921201 0.559507421379071 0.518589386631407; visual box size=0.8312712463921201 0.559507421379071 0.518589386631407
- added link link5NNP, mass 1; collision box size=0.4115067271500367 0.31856623679810997 0.8513225167663709; visual box size=0.4115067271500367 0.31856623679810997 0.8513225167663709
- added link link5NPP, mass 1; collision box size=0.4115067271500367 0.31856623679810997 0.8513225167663709; visual box size=0.4115067271500367 0.31856623679810997 0.8513225167663709
- link link2NNP: geometry collision box size=0.2096368522853158 0.5654848559859877 0.5701950169606016; visual box size=0.2096368522853158 0.5654848559859877 0.5701950169606016
- link link2NPP: geometry collision box size=0.2096368522853158 0.5654848559859877 0.5701950169606016; visual box size=0.2096368522853158 0.5654848559859877 0.5701950169606016
- link link3NNP: geometry collision box size=0.5509384984747858 0.42437023576917177 0.8033612530830243; visual box size=0.5509384984747858 0.42437023576917177 0.8033612530830243
- link link3NPP: geometry collision box size=0.5509384984747858 0.42437023576917177 0.8033612530830243; visual box size=0.5509384984747858 0.42437023576917177 0.8033612530830243
Joints:
- added joint link3NNP_link4NNP: type revolute, parent link3NNP, child link4NNP, origin xyz=0 -0.21218511788458588 0.40168062654151215 rpy=0 0 0, axis 0 1 0, limit lower=-3.14159 upper=3.14159 effort=0.0 velocity=0.0
- added joint link3NPP_link4NPP: type revolute, parent link3NPP, child link4NPP, origin xyz=0 0.21218511788458588 0.40168062654151215 rpy=0 0 0, axis 0 1 0, limit lower=-3.14159 upper=3.14159 effort=0.0 velocity=0.0
- added joint link4NNP_link5NNP: type revolute, parent link4NNP, child link5NNP, origin xyz=0 -0.2797537106895355 0.2592946933157035 rpy=0 0 0, axis 0 1 0, limit lower=-3.14159 upper=3.14159 effort=0.0 velocity=0.0
- added joint link4NPP_link5NPP: type revolute, parent link4NPP, child link5NPP, origin xyz=0 0.2797537106895355 0.2592946933157035 rpy=0 0 0, axis 0 1 0, limit lower=-3.14159 upper=3.14159 effort=0.0 velocity=0.0
- joint link1NNP_link2NNP: origin xyz=0 0.0 0.5 rpy=0 0 0 -> xyz=0.0 0 0.5 rpy=0 0 0
- joint link1NPP_link2NPP: origin xyz=0 0.0 0.5 rpy=0 0 0 -> xyz=0.0 0 0.5 rpy=0 0 0
- joint link2NNP_link3NNP: axis 0 1 0 -> 0 0 1; origin xyz=0 -0.25729393851084215 0.17709900065518247 rpy=0 0 0 -> xyz=-0.1048184261426579 0 0.2850975084803008 rpy=0 0 0
- joint link2NPP_link3NPP: axis 0 1 0 -> 0 0 1; origin xyz=0 0.25729393851084215 0.17709900065518247 rpy=0 0 0 -> xyz=-0.1048184261426579 0 0.2850975084803008 rpy=0 0 0

File: body6.urdf (robot description, URDF)
Before this commit: robot robot, 13 links, 12 joints
Links:
- removed link link6NNP
- removed link link6NPP
- link link2NNP: geometry collision box size=0.2096368522853158 0.5654848559859877 0.5701950169606016; visual box size=0.2096368522853158 0.5654848559859877 0.5701950169606016
- link link2NPP: geometry collision box size=0.2096368522853158 0.5654848559859877 0.5701950169606016; visual box size=0.2096368522853158 0.5654848559859877 0.5701950169606016
- link link3NNP: geometry collision box size=0.5509384984747858 0.42437023576917177 0.8033612530830243; visual box size=0.5509384984747858 0.42437023576917177 0.8033612530830243
- link link3NPP: geometry collision box size=0.5509384984747858 0.42437023576917177 0.8033612530830243; visual box size=0.5509384984747858 0.42437023576917177 0.8033612530830243
- link link4NNP: geometry collision box size=0.8312712463921201 0.559507421379071 0.518589386631407; visual box size=0.8312712463921201 0.559507421379071 0.518589386631407
- link link4NPP: geometry collision box size=0.8312712463921201 0.559507421379071 0.518589386631407; visual box size=0.8312712463921201 0.559507421379071 0.518589386631407
- link link5NNP: geometry collision box size=0.4115067271500367 0.31856623679810997 0.8513225167663709; visual box size=0.4115067271500367 0.31856623679810997 0.8513225167663709
- link link5NPP: geometry collision box size=0.4115067271500367 0.31856623679810997 0.8513225167663709; visual box size=0.4115067271500367 0.31856623679810997 0.8513225167663709
Joints:
- removed joint link5NNP_link6NNP
- removed joint link5NPP_link6NPP
- joint link1NNP_link2NNP: origin xyz=0 0.0 0.5 rpy=0 0 0 -> xyz=0.0 0 0.5 rpy=0 0 0
- joint link1NPP_link2NPP: origin xyz=0 0.0 0.5 rpy=0 0 0 -> xyz=0.0 0 0.5 rpy=0 0 0
- joint link2NNP_link3NNP: axis 1 0 0 -> 0 1 0; origin xyz=-0.4226763108474717 -0.29209895486477533 0 rpy=0 0 0 -> xyz=-0.1048184261426579 0 0.2850975084803008 rpy=0 0 0
- joint link2NPP_link3NPP: axis 1 0 0 -> 0 1 0; origin xyz=-0.4226763108474717 0.29209895486477533 0 rpy=0 0 0 -> xyz=-0.1048184261426579 0 0.2850975084803008 rpy=0 0 0
- joint link3NNP_link4NNP: axis 0 0 1 -> 0 1 0; origin xyz=-0.14406481956688474 0 0.25366844181771897 rpy=0 0 0 -> xyz=0 -0.21218511788458588 0.40168062654151215 rpy=0 0 0
- joint link3NPP_link4NPP: axis 0 0 1 -> 0 1 0; origin xyz=-0.14406481956688474 0 0.25366844181771897 rpy=0 0 0 -> xyz=0 0.21218511788458588 0.40168062654151215 rpy=0 0 0
- joint link4NNP_link5NNP: origin xyz=0 -0.20032053411360673 0.2269740362182999 rpy=0 0 0 -> xyz=0 -0.2797537106895355 0.2592946933157035 rpy=0 0 0
- joint link4NPP_link5NPP: origin xyz=0 0.20032053411360673 0.2269740362182999 rpy=0 0 0 -> xyz=0 0.2797537106895355 0.2592946933157035 rpy=0 0 0

File: body7.urdf (robot description, URDF)
Before this commit: robot robot, 9 links, 8 joints
Links:
- added link link5NNP, mass 1; collision box size=0.4115067271500367 0.31856623679810997 0.8513225167663709; visual box size=0.4115067271500367 0.31856623679810997 0.8513225167663709
- added link link5NPP, mass 1; collision box size=0.4115067271500367 0.31856623679810997 0.8513225167663709; visual box size=0.4115067271500367 0.31856623679810997 0.8513225167663709
- link link2NNP: geometry collision box size=0.2096368522853158 0.5654848559859877 0.5701950169606016; visual box size=0.2096368522853158 0.5654848559859877 0.5701950169606016
- link link2NPP: geometry collision box size=0.2096368522853158 0.5654848559859877 0.5701950169606016; visual box size=0.2096368522853158 0.5654848559859877 0.5701950169606016
- link link3NNP: geometry collision box size=0.5509384984747858 0.42437023576917177 0.8033612530830243; visual box size=0.5509384984747858 0.42437023576917177 0.8033612530830243
- link link3NPP: geometry collision box size=0.5509384984747858 0.42437023576917177 0.8033612530830243; visual box size=0.5509384984747858 0.42437023576917177 0.8033612530830243
- link link4NNP: geometry collision box size=0.8312712463921201 0.559507421379071 0.518589386631407; visual box size=0.8312712463921201 0.559507421379071 0.518589386631407
- link link4NPP: geometry collision box size=0.8312712463921201 0.559507421379071 0.518589386631407; visual box size=0.8312712463921201 0.559507421379071 0.518589386631407
Joints:
- added joint link4NNP_link5NNP: type revolute, parent link4NNP, child link5NNP, origin xyz=0 -0.2797537106895355 0.2592946933157035 rpy=0 0 0, axis 0 1 0, limit lower=-3.14159 upper=3.14159 effort=0.0 velocity=0.0
- added joint link4NPP_link5NPP: type revolute, parent link4NPP, child link5NPP, origin xyz=0 0.2797537106895355 0.2592946933157035 rpy=0 0 0, axis 0 1 0, limit lower=-3.14159 upper=3.14159 effort=0.0 velocity=0.0
- joint link1NNP_link2NNP: origin xyz=0 0.0 0.5 rpy=0 0 0 -> xyz=0.0 0 0.5 rpy=0 0 0
- joint link1NPP_link2NPP: origin xyz=0 0.0 0.5 rpy=0 0 0 -> xyz=0.0 0 0.5 rpy=0 0 0
- joint link2NNP_link3NNP: origin xyz=0 -0.20145771345462804 0.44349343321948786 rpy=0 0 0 -> xyz=-0.1048184261426579 0 0.2850975084803008 rpy=0 0 0
- joint link2NPP_link3NPP: origin xyz=0 0.20145771345462804 0.44349343321948786 rpy=0 0 0 -> xyz=-0.1048184261426579 0 0.2850975084803008 rpy=0 0 0
- joint link3NNP_link4NNP: axis 1 0 0 -> 0 1 0; origin xyz=0 -0.18173481049146967 0.30242802774898714 rpy=0 0 0 -> xyz=0 -0.21218511788458588 0.40168062654151215 rpy=0 0 0
- joint link3NPP_link4NPP: axis 1 0 0 -> 0 1 0; origin xyz=0 0.18173481049146967 0.30242802774898714 rpy=0 0 0 -> xyz=0 0.21218511788458588 0.40168062654151215 rpy=0 0 0

File: body8.urdf (robot description, URDF)
Before this commit: robot robot, 9 links, 8 joints
Links:
- added link link5NNP, mass 1; collision box size=0.4115067271500367 0.31856623679810997 0.8513225167663709; visual box size=0.4115067271500367 0.31856623679810997 0.8513225167663709
- added link link5NPP, mass 1; collision box size=0.4115067271500367 0.31856623679810997 0.8513225167663709; visual box size=0.4115067271500367 0.31856623679810997 0.8513225167663709
- link link2NNP: geometry collision box size=0.2096368522853158 0.5654848559859877 0.5701950169606016; visual box size=0.2096368522853158 0.5654848559859877 0.5701950169606016
- link link2NPP: geometry collision box size=0.2096368522853158 0.5654848559859877 0.5701950169606016; visual box size=0.2096368522853158 0.5654848559859877 0.5701950169606016
- link link3NNP: geometry collision box size=0.5509384984747858 0.42437023576917177 0.8033612530830243; visual box size=0.5509384984747858 0.42437023576917177 0.8033612530830243
- link link3NPP: geometry collision box size=0.5509384984747858 0.42437023576917177 0.8033612530830243; visual box size=0.5509384984747858 0.42437023576917177 0.8033612530830243
- link link4NNP: geometry collision box size=0.8312712463921201 0.559507421379071 0.518589386631407; visual box size=0.8312712463921201 0.559507421379071 0.518589386631407
- link link4NPP: geometry collision box size=0.8312712463921201 0.559507421379071 0.518589386631407; visual box size=0.8312712463921201 0.559507421379071 0.518589386631407
Joints:
- added joint link4NNP_link5NNP: type revolute, parent link4NNP, child link5NNP, origin xyz=0 -0.2797537106895355 0.2592946933157035 rpy=0 0 0, axis 0 1 0, limit lower=-3.14159 upper=3.14159 effort=0.0 velocity=0.0
- added joint link4NPP_link5NPP: type revolute, parent link4NPP, child link5NPP, origin xyz=0 0.2797537106895355 0.2592946933157035 rpy=0 0 0, axis 0 1 0, limit lower=-3.14159 upper=3.14159 effort=0.0 velocity=0.0
- joint link1NNP_link2NNP: origin xyz=0 0.0 0.5 rpy=0 0 0 -> xyz=0.0 0 0.5 rpy=0 0 0
- joint link1NPP_link2NPP: origin xyz=0 0.0 0.5 rpy=0 0 0 -> xyz=0.0 0 0.5 rpy=0 0 0
- joint link2NNP_link3NNP: origin xyz=0 -0.25729393851084215 0.17709900065518247 rpy=0 0 0 -> xyz=-0.1048184261426579 0 0.2850975084803008 rpy=0 0 0
- joint link2NPP_link3NPP: origin xyz=0 0.25729393851084215 0.17709900065518247 rpy=0 0 0 -> xyz=-0.1048184261426579 0 0.2850975084803008 rpy=0 0 0
- joint link3NNP_link4NNP: axis 0 0 1 -> 0 1 0; origin xyz=-0.20006888407041173 0 0.23912862336301505 rpy=0 0 0 -> xyz=0 -0.21218511788458588 0.40168062654151215 rpy=0 0 0
- joint link3NPP_link4NPP: axis 0 0 1 -> 0 1 0; origin xyz=-0.20006888407041173 0 0.23912862336301505 rpy=0 0 0 -> xyz=0 0.21218511788458588 0.40168062654151215 rpy=0 0 0

File: body9.urdf (robot description, URDF)
Before this commit: robot robot, 13 links, 12 joints
Links:
- removed link link6NNP
- removed link link6NPP
- link link2NNP: geometry collision box size=0.2096368522853158 0.5654848559859877 0.5701950169606016; visual box size=0.2096368522853158 0.5654848559859877 0.5701950169606016
- link link2NPP: geometry collision box size=0.2096368522853158 0.5654848559859877 0.5701950169606016; visual box size=0.2096368522853158 0.5654848559859877 0.5701950169606016
- link link3NNP: geometry collision box size=0.5509384984747858 0.42437023576917177 0.8033612530830243; visual box size=0.5509384984747858 0.42437023576917177 0.8033612530830243
- link link3NPP: geometry collision box size=0.5509384984747858 0.42437023576917177 0.8033612530830243; visual box size=0.5509384984747858 0.42437023576917177 0.8033612530830243
- link link4NNP: geometry collision box size=0.8312712463921201 0.559507421379071 0.518589386631407; visual box size=0.8312712463921201 0.559507421379071 0.518589386631407
- link link4NPP: geometry collision box size=0.8312712463921201 0.559507421379071 0.518589386631407; visual box size=0.8312712463921201 0.559507421379071 0.518589386631407
- link link5NNP: geometry collision box size=0.4115067271500367 0.31856623679810997 0.8513225167663709; visual box size=0.4115067271500367 0.31856623679810997 0.8513225167663709
- link link5NPP: geometry collision box size=0.4115067271500367 0.31856623679810997 0.8513225167663709; visual box size=0.4115067271500367 0.31856623679810997 0.8513225167663709
Joints:
- removed joint link5NNP_link6NNP
- removed joint link5NPP_link6NPP
- joint link1NNP_link2NNP: origin xyz=0 0.0 0.5 rpy=0 0 0 -> xyz=0.0 0 0.5 rpy=0 0 0
- joint link1NPP_link2NPP: origin xyz=0 0.0 0.5 rpy=0 0 0 -> xyz=0.0 0 0.5 rpy=0 0 0
- joint link2NNP_link3NNP: axis 1 0 0 -> 0 1 0; origin xyz=-0.4226763108474717 -0.29209895486477533 0 rpy=0 0 0 -> xyz=-0.1048184261426579 0 0.2850975084803008 rpy=0 0 0
- joint link2NPP_link3NPP: axis 1 0 0 -> 0 1 0; origin xyz=-0.4226763108474717 0.29209895486477533 0 rpy=0 0 0 -> xyz=-0.1048184261426579 0 0.2850975084803008 rpy=0 0 0
- joint link3NNP_link4NNP: origin xyz=-0.14406481956688474 0 0.25366844181771897 rpy=0 0 0 -> xyz=0 -0.21218511788458588 0.40168062654151215 rpy=0 0 0
- joint link3NPP_link4NPP: origin xyz=-0.14406481956688474 0 0.25366844181771897 rpy=0 0 0 -> xyz=0 0.21218511788458588 0.40168062654151215 rpy=0 0 0
- joint link4NNP_link5NNP: origin xyz=0 -0.20032053411360673 0.2269740362182999 rpy=0 0 0 -> xyz=0 -0.2797537106895355 0.2592946933157035 rpy=0 0 0
- joint link4NPP_link5NPP: origin xyz=0 0.20032053411360673 0.2269740362182999 rpy=0 0 0 -> xyz=0 0.2797537106895355 0.2592946933157035 rpy=0 0 0

Commit message: FP: checking on plots

File: body0.urdf (robot description, URDF)
Before this commit: robot robot, 9 links, 8 joints
Links:
- removed link link4NNP
- removed link link4NPP
- link link2NNP: geometry collision box size=0.4426388687084081 0.4884867620350666 0.5831027159391181; visual box size=0.4426388687084081 0.4884867620350666 0.5831027159391181
- link link2NPP: geometry collision box size=0.4426388687084081 0.4884867620350666 0.5831027159391181; visual box size=0.4426388687084081 0.4884867620350666 0.5831027159391181
- link link3NNP: geometry collision box size=0.25321207654367195 0.36063640579402995 0.9343640344701751; visual box size=0.25321207654367195 0.36063640579402995 0.9343640344701751
- link link3NPP: geometry collision box size=0.25321207654367195 0.36063640579402995 0.9343640344701751; visual box size=0.25321207654367195 0.36063640579402995 0.9343640344701751
Joints:
- removed joint link3NNP_link4NNP
- removed joint link3NPP_link4NPP
- joint link1NNP_link2NNP: origin xyz=0 0.0 0.5 rpy=0 0 0 -> xyz=0.0 0 0.5 rpy=0 0 0
- joint link1NPP_link2NPP: origin xyz=0 0.0 0.5 rpy=0 0 0 -> xyz=0.0 0 0.5 rpy=0 0 0
- joint link2NNP_link3NNP: axis 0 0 1 -> 1 0 0; origin xyz=-0.40318176117612103 -0.184114316166169 0 rpy=0 0 0 -> xyz=-0.22131943435420404 0 0.29155135796955906 rpy=0 0 0
- joint link2NPP_link3NPP: axis 0 0 1 -> 1 0 0; origin xyz=-0.40318176117612103 0.184114316166169 0 rpy=0 0 0 -> xyz=-0.22131943435420404 0 0.29155135796955906 rpy=0 0 0

File: body1.urdf (robot description, URDF)
Before this commit: robot robot, 9 links, 8 joints
Links:
- removed link link4NNP
- removed link link4NPP
- link link2NNP: geometry collision box size=0.4426388687084081 0.4884867620350666 0.5831027159391181; visual box size=0.4426388687084081 0.4884867620350666 0.5831027159391181
- link link2NPP: geometry collision box size=0.4426388687084081 0.4884867620350666 0.5831027159391181; visual box size=0.4426388687084081 0.4884867620350666 0.5831027159391181
- link link3NNP: geometry collision box size=0.25321207654367195 0.36063640579402995 0.9343640344701751; visual box size=0.25321207654367195 0.36063640579402995 0.9343640344701751
- link link3NPP: geometry collision box size=0.25321207654367195 0.36063640579402995 0.9343640344701751; visual box size=0.25321207654367195 0.36063640579402995 0.9343640344701751
Joints:
- removed joint link3NNP_link4NNP
- removed joint link3NPP_link4NPP
- joint link1NNP_link2NNP: origin xyz=0 0.0 0.5 rpy=0 0 0 -> xyz=0.0 0 0.5 rpy=0 0 0
- joint link1NPP_link2NPP: origin xyz=0 0.0 0.5 rpy=0 0 0 -> xyz=0.0 0 0.5 rpy=0 0 0
- joint link2NNP_link3NNP: axis 0 0 1 -> 1 0 0; origin xyz=-0.40318176117612103 -0.184114316166169 0 rpy=0 0 0 -> xyz=-0.22131943435420404 0 0.29155135796955906 rpy=0 0 0
- joint link2NPP_link3NPP: axis 0 0 1 -> 1 0 0; origin xyz=-0.40318176117612103 0.184114316166169 0 rpy=0 0 0 -> xyz=-0.22131943435420404 0 0.29155135796955906 rpy=0 0 0

Commit message: FP: fixed random seeds and added experimental data files

File: body0.urdf (robot description, URDF)
Before this commit: robot robot, 7 links, 6 joints
Links:
- added link link4NNP, mass 1; collision box size=0.48643949975599066 0.556664263928273 0.37475418153218537; visual box size=0.48643949975599066 0.556664263928273 0.37475418153218537
- added link link4NPP, mass 1; collision box size=0.48643949975599066 0.556664263928273 0.37475418153218537; visual box size=0.48643949975599066 0.556664263928273 0.37475418153218537
- link link2NNP: geometry collision box size=0.8063635223522421 0.368228632332338 0.4071334002343707; visual box size=0.8063635223522421 0.368228632332338 0.4071334002343707
- link link2NPP: geometry collision box size=0.8063635223522421 0.368228632332338 0.4071334002343707; visual box size=0.8063635223522421 0.368228632332338 0.4071334002343707
- link link3NNP: geometry collision box size=0.5239473099603315 0.513519435613909 0.442650180863142; visual box size=0.5239473099603315 0.513519435613909 0.442650180863142
- link link3NPP: geometry collision box size=0.5239473099603315 0.513519435613909 0.442650180863142; visual box size=0.5239473099603315 0.513519435613909 0.442650180863142
Joints:
- added joint link3NNP_link4NNP: type revolute, parent link3NNP, child link4NNP, origin xyz=-0.2619736549801657 0 0.221325090431571 rpy=0 0 0, axis 0 0 1, limit lower=-3.14159 upper=3.14159 effort=0.0 velocity=0.0
- added joint link3NPP_link4NPP: type revolute, parent link3NPP, child link4NPP, origin xyz=-0.2619736549801657 0 0.221325090431571 rpy=0 0 0, axis 0 0 1, limit lower=-3.14159 upper=3.14159 effort=0.0 velocity=0.0
- joint link1NNP_link2NNP: origin xyz=0.0 0 0.5 rpy=0 0 0 -> xyz=0 0.0 0.5 rpy=0 0 0
- joint link1NPP_link2NPP: origin xyz=0.0 0 0.5 rpy=0 0 0 -> xyz=0 0.0 0.5 rpy=0 0 0
- joint link2NNP_link3NNP: axis 1 0 0 -> 0 0 1; origin xyz=-0.22131943435420404 0 0.29155135796955906 rpy=0 0 0 -> xyz=-0.40318176117612103 -0.184114316166169 0 rpy=0 0 0
- joint link2NPP_link3NPP: axis 1 0 0 -> 0 0 1; origin xyz=-0.22131943435420404 0 0.29155135796955906 rpy=0 0 0 -> xyz=-0.40318176117612103 0.184114316166169 0 rpy=0 0 0

File: body1.urdf (robot description, URDF)
Before this commit: robot robot, 7 links, 6 joints
Links:
- added link link4NNP, mass 1; collision box size=0.48643949975599066 0.556664263928273 0.37475418153218537; visual box size=0.48643949975599066 0.556664263928273 0.37475418153218537
- added link link4NPP, mass 1; collision box size=0.48643949975599066 0.556664263928273 0.37475418153218537; visual box size=0.48643949975599066 0.556664263928273 0.37475418153218537
- link link2NNP: geometry collision box size=0.8063635223522421 0.368228632332338 0.4071334002343707; visual box size=0.8063635223522421 0.368228632332338 0.4071334002343707
- link link2NPP: geometry collision box size=0.8063635223522421 0.368228632332338 0.4071334002343707; visual box size=0.8063635223522421 0.368228632332338 0.4071334002343707
- link link3NNP: geometry collision box size=0.5239473099603315 0.513519435613909 0.442650180863142; visual box size=0.5239473099603315 0.513519435613909 0.442650180863142
- link link3NPP: geometry collision box size=0.5239473099603315 0.513519435613909 0.442650180863142; visual box size=0.5239473099603315 0.513519435613909 0.442650180863142
Joints:
- added joint link3NNP_link4NNP: type revolute, parent link3NNP, child link4NNP, origin xyz=-0.2619736549801657 0 0.221325090431571 rpy=0 0 0, axis 0 0 1, limit lower=-3.14159 upper=3.14159 effort=0.0 velocity=0.0
- added joint link3NPP_link4NPP: type revolute, parent link3NPP, child link4NPP, origin xyz=-0.2619736549801657 0 0.221325090431571 rpy=0 0 0, axis 0 0 1, limit lower=-3.14159 upper=3.14159 effort=0.0 velocity=0.0
- joint link1NNP_link2NNP: origin xyz=0.0 0 0.5 rpy=0 0 0 -> xyz=0 0.0 0.5 rpy=0 0 0
- joint link1NPP_link2NPP: origin xyz=0.0 0 0.5 rpy=0 0 0 -> xyz=0 0.0 0.5 rpy=0 0 0
- joint link2NNP_link3NNP: axis 1 0 0 -> 0 0 1; origin xyz=-0.22131943435420404 0 0.29155135796955906 rpy=0 0 0 -> xyz=-0.40318176117612103 -0.184114316166169 0 rpy=0 0 0
- joint link2NPP_link3NPP: axis 1 0 0 -> 0 0 1; origin xyz=-0.22131943435420404 0 0.29155135796955906 rpy=0 0 0 -> xyz=-0.40318176117612103 0.184114316166169 0 rpy=0 0 0
