Commit message: FP: playing with mutation function

File: body0.urdf (robot description, URDF)
Before this commit: robot robot, 7 links, 6 joints
Links:
- removed link link3NNP
- removed link link3NPP
- link link2NNP: geometry collision box size=0.4426388687084081 0.4884867620350666 0.5831027159391181; visual box size=0.4426388687084081 0.4884867620350666 0.5831027159391181
- link link2NPP: geometry collision box size=0.4426388687084081 0.4884867620350666 0.5831027159391181; visual box size=0.4426388687084081 0.4884867620350666 0.5831027159391181
Joints:
- removed joint link2NNP_link3NNP
- removed joint link2NPP_link3NPP
- joint link1NNP_link2NNP: origin xyz=0.0 0 0.5 rpy=0 0 0 -> xyz=0 0.0 0.5 rpy=0 0 0
- joint link1NPP_link2NPP: origin xyz=0.0 0 0.5 rpy=0 0 0 -> xyz=0 0.0 0.5 rpy=0 0 0

File: body1.urdf (robot description, URDF)
Before this commit: robot robot, 9 links, 8 joints
Links:
- removed link link4NNP
- removed link link4NPP
- link link2NNP: geometry collision box size=0.4426388687084081 0.4884867620350666 0.5831027159391181; visual box size=0.4426388687084081 0.4884867620350666 0.5831027159391181
- link link2NPP: geometry collision box size=0.4426388687084081 0.4884867620350666 0.5831027159391181; visual box size=0.4426388687084081 0.4884867620350666 0.5831027159391181
- link link3NNP: geometry collision box size=0.25321207654367195 0.36063640579402995 0.9343640344701751; visual box size=0.25321207654367195 0.36063640579402995 0.9343640344701751
- link link3NPP: geometry collision box size=0.25321207654367195 0.36063640579402995 0.9343640344701751; visual box size=0.25321207654367195 0.36063640579402995 0.9343640344701751
Joints:
- removed joint link3NNP_link4NNP
- removed joint link3NPP_link4NPP
- joint link1NNP_link2NNP: origin xyz=0.0 0 0.5 rpy=0 0 0 -> xyz=0 0.0 0.5 rpy=0 0 0
- joint link1NPP_link2NPP: origin xyz=0.0 0 0.5 rpy=0 0 0 -> xyz=0 0.0 0.5 rpy=0 0 0
- joint link2NNP_link3NNP: origin xyz=-0.33705636425086627 -0.12608455921702855 0 rpy=0 0 0 -> xyz=-0.22131943435420404 -0.2442433810175333 0 rpy=0 0 0
- joint link2NPP_link3NPP: origin xyz=-0.33705636425086627 0.12608455921702855 0 rpy=0 0 0 -> xyz=-0.22131943435420404 0.2442433810175333 0 rpy=0 0 0

Commit message: FP: working through stuff

File: body0.urdf (robot description, URDF)
Before this commit: robot robot, 5 links, 4 joints
Links:
- added link link3NNP, mass 1; collision box size=0.6213375018146079 0.4786906808847609 0.8819849749885769; visual box size=0.6213375018146079 0.4786906808847609 0.8819849749885769
- added link link3NPP, mass 1; collision box size=0.6213375018146079 0.4786906808847609 0.8819849749885769; visual box size=0.6213375018146079 0.4786906808847609 0.8819849749885769
- link link2NNP: geometry collision box size=0.9789781879753565 0.3331232246829251 0.3479846634002767; visual box size=0.9789781879753565 0.3331232246829251 0.3479846634002767
- link link2NPP: geometry collision box size=0.9789781879753565 0.3331232246829251 0.3479846634002767; visual box size=0.9789781879753565 0.3331232246829251 0.3479846634002767
Joints:
- added joint link2NNP_link3NNP: type revolute, parent link2NNP, child link3NNP, origin xyz=-0.48948909398767826 -0.16656161234146255 0 rpy=0 0 0, axis 0 0 1, limit lower=-3.14159 upper=3.14159 effort=0.0 velocity=0.0
- added joint link2NPP_link3NPP: type revolute, parent link2NPP, child link3NPP, origin xyz=-0.48948909398767826 0.16656161234146255 0 rpy=0 0 0, axis 0 0 1, limit lower=-3.14159 upper=3.14159 effort=0.0 velocity=0.0

File: body2.urdf (robot description, URDF)
Before this commit: robot robot, 7 links, 6 joints
Links:
- added link link4NNP, mass 1; collision box size=0.30840537681640073 0.5966962336065149 0.29789516740030736; visual box size=0.30840537681640073 0.5966962336065149 0.29789516740030736
- added link link4NPP, mass 1; collision box size=0.30840537681640073 0.5966962336065149 0.29789516740030736; visual box size=0.30840537681640073 0.5966962336065149 0.29789516740030736
Joints:
- added joint link3NNP_link4NNP: type revolute, parent link3NNP, child link4NNP, origin xyz=-0.31066875090730395 -0.23934534044238046 0 rpy=0 0 0, axis 1 0 0, limit lower=-3.14159 upper=3.14159 effort=0.0 velocity=0.0
- added joint link3NPP_link4NPP: type revolute, parent link3NPP, child link4NPP, origin xyz=-0.31066875090730395 0.23934534044238046 0 rpy=0 0 0, axis 1 0 0, limit lower=-3.14159 upper=3.14159 effort=0.0 velocity=0.0
